File: Keyboard_PCB/keyboard_schematic.sch (EAGLE design)
At the start: 3 parts

Commit message: Added parts
Parts:
- added 0, 1, 2, 3, 4, 5, 6, 7, 8, 9, A, ALT, ALT2, B, BACKSLASH, BACKSONG, BACKSPACE_1, C, CAPSLOCK, COMMA, CTRL, CTRL2, D, DASH, DELETE, DELETE2, DOWN, E, END, ENTER2, EQUAL, EQUAL2, F, F10, F11, F12, F3, F4, F5, F6, F7, F8, F9, G, GRAVE, H, HOME, I, INSERT, J, K, KP_1, KP_2, KP_3, KP_4, KP_5, KP_52, KP_6, KP_62, KP_7, KP_8, KP_9, KP_ASTERISK, KP_DASH, KP_DEL, KP_SLASH, L, LBRACKET, LEFT, M, MENU, N, NEXTSONG, NUMLOCK, O, P, PAUSE, PAUSEPLAY, PERIOD, PGDN, PGUP, PRTSC, Q, QUOTE, R, RANDSONG, RBRACKET, RIGHT, S, SCROLLLOCK, SEMICOLON, SLASH, T, TAB, U, UNDERSCORE, UP, V, VOLUMEUP, VOLUMNEDOWN, W, WIN, WIN2, X, Y, Z: KEYSWITCH-RGBLED-MX-1U-RGB, Keyboard:KEYSWITCH-RGBLED-MX-1U-RGB
- added BACKSPACE, ENTER, KP_0, SHIFT, SHIFT2: KEYSWITCH-RGBLED-MX-2U-RGB, Keyboard:KEYSWITCH-RGBLED-MX-2U-RGB
- added D0, D1, D2, D3, D4, D5, D6, D7, D8, D9, DA, DALT, DALT2, DB, DBACKSLASH, DBACKSONG, DBACKSPACE, DBACKSPACE_1, DC, DCAPSLOCK, DCOMMA, DCTRL, DCTRL2, DD, DDASH, DDELETE, DDELETE2, DDOWN, DE, DEND, DENTER, DENTER2, DEQUAL, DEQUAL2, DESC, DF, DF1, DF10, DF11, DF12, DF2, DF3, DF4, DF5, DF6, DF7, DF8, DF9, DG, DGRAVE, DH, DHOME, DI, DINSERT, DJ, DK, DKP_0, DKP_1, DKP_2, DKP_3, DKP_4, DKP_5, DKP_52, DKP_6, DKP_62, DKP_7, DKP_8, DKP_9, DKP_ASTERISK, DKP_DASH, DKP_DEL, DKP_SLASH, DL, DLBRACKET, DLEFT, DM, DMENU, DN, DNEXTSONG, DNUMLOCK, DO, DP, DPAUSE, DPAUSEPLAY, DPERIOD, DPGDN, DPGUP, DPRTSC, DQ, DQUOTE, DR, DRANDSONG, DRBRACKET, DRIGHT, DS, DSCROLLLOCK, DSEMICOLON, DSHIFT, DSHIFT2, DSLASH, DSPACE, DT, DTAB, DU, DUNDERSCORE, DUP, DV, DVOLUMEUP, DVOLUMNEDOWN, DW, DWIN, DWIN2, DX, DY, DZ: 1N4148, Components:DIODE-DO-35
- added SPACE: KEYSWITCH-RGBLED-MX-6.25U-RGB, Keyboard:KEYSWITCH-RGBLED-MX-6.25U-RGB
Connections:
- new net ROW1.5: DBACKSONG.C, DESC.C, DF1.C, DF10.C, DF11.C, DF12.C, DF2.C, DF3.C, DF4.C, DF5.C, DF6.C, DF7.C, DF8.C, DF9.C, DNEXTSONG.C, DPAUSE.C, DPAUSEPLAY.C, DPRTSC.C, DRANDSONG.C, DSCROLLLOCK.C, DVOLUMEUP.C, DVOLUMNEDOWN.C
- new net ROW2.5: D0.C, D1.C, D2.C, D3.C, D4.C, D5.C, D6.C, D7.C, D8.C, D9.C, DBACKSPACE.C, DDASH.C, DEQUAL.C, DGRAVE.C, DHOME.C, DINSERT.C, DKP_ASTERISK.C, DKP_DASH.C, DKP_SLASH.C, DNUMLOCK.C, DPGUP.C, DUNDERSCORE.C
- new net ROW3.5: DBACKSLASH.C, DDELETE.C, DE.C, DEND.C, DI.C, DKP_7.C, DKP_8.C, DKP_9.C, DLBRACKET.C, DO.C, DP.C, DPGDN.C, DQ.C, DR.C, DRBRACKET.C, DT.C, DTAB.C, DU.C, DW.C, DY.C
- new net ROW4.5: DA.C, DCAPSLOCK.C, DD.C, DENTER.C, DF.C, DG.C, DH.C, DJ.C, DK.C, DKP_4.C, DKP_52.C, DKP_6.C, DKP_62.C, DL.C, DQUOTE.C, DS.C, DSEMICOLON.C
- new net ROW5.5: DB.C, DC.C, DCOMMA.C, DKP_1.C, DKP_2.C, DKP_3.C, DM.C, DN.C, DPERIOD.C, DSHIFT.C, DSHIFT2.C, DSLASH.C, DUP.C, DV.C, DX.C, DZ.C
- new net ROW6.5: DALT.C, DALT2.C, DBACKSPACE_1.C, DCTRL.C, DCTRL2.C, DDOWN.C, DKP_0.C, DKP_DEL.C, DLEFT.C, DMENU.C, DRIGHT.C, DSPACE.C, DWIN.C, DWIN2.C

Commit message: Updated Schematic
Parts:
- removed 0, 1, 2, 3, 4, 5, 6, 7, 8, 9, A, ALT, ALT2, B, BACKSLASH, BACKSONG, BACKSPACE_1, C, CAPSLOCK, COMMA, CTRL, CTRL2, D, DASH, DELETE, DELETE2, DOWN, E, END, ENTER2, EQUAL, EQUAL2, ESC, F, F1, F10, F11, F12, F2, F3, F4, F5, F6, F7, F8, F9, G, GRAVE, H, HOME, I, INSERT, J, K, KP_1, KP_2, KP_3, KP_4, KP_5, KP_52, KP_6, KP_62, KP_7, KP_8, KP_9, KP_ASTERISK, KP_DASH, KP_DEL, KP_SLASH, L, LBRACKET, LEFT, M, MENU, N, NEXTSONG, NUMLOCK, O, P, PAUSE, PAUSEPLAY, PERIOD, PGDN, PGUP, PRTSC, Q, QUOTE, R, RANDSONG, RBRACKET, RIGHT, S, SCROLLLOCK, SEMICOLON, SLASH, T, TAB, U, UNDERSCORE, UP, V, VOLUMEUP, VOLUMNEDOWN, W, WIN, WIN2, X, Y, Z: KEYSWITCH-RGBLED-MX-1U-RGB, Keyboard:KEYSWITCH-RGBLED-MX-1U-RGB
- removed BACKSPACE, ENTER, KP_0, SHIFT, SHIFT2: KEYSWITCH-RGBLED-MX-2U-RGB, Keyboard:KEYSWITCH-RGBLED-MX-2U-RGB
- removed D0, D1, D2, D3, D4, D5, D6, D7, D8, D9, DA, DALT, DALT2, DB, DBACKSLASH, DBACKSONG, DBACKSPACE, DBACKSPACE_1, DC, DCAPSLOCK, DCOMMA, DCTRL, DCTRL2, DD, DDASH, DDELETE, DDELETE2, DDOWN, DE, DEND, DENTER, DENTER2, DEQUAL, DEQUAL2, DESC, DF, DF1, DF10, DF11, DF12, DF2, DF3, DF4, DF5, DF6, DF7, DF8, DF9, DG, DGRAVE, DH, DHOME, DI, DINSERT, DJ, DK, DKP_0, DKP_1, DKP_2, DKP_3, DKP_4, DKP_5, DKP_52, DKP_6, DKP_62, DKP_7, DKP_8, DKP_9, DKP_ASTERISK, DKP_DASH, DKP_DEL, DKP_SLASH, DL, DLBRACKET, DLEFT, DM, DMENU, DN, DNEXTSONG, DNUMLOCK, DO, DP, DPAUSE, DPAUSEPLAY, DPERIOD, DPGDN, DPGUP, DPRTSC, DQ, DQUOTE, DR, DRANDSONG, DRBRACKET, DRIGHT, DS, DSCROLLLOCK, DSEMICOLON, DSHIFT, DSHIFT2, DSLASH, DSPACE, DT, DTAB, DU, DUNDERSCORE, DUP, DV, DVOLUMEUP, DVOLUMNEDOWN, DW, DWIN, DWIN2, DX, DY, DZ: 1N4148, Components:DIODE-DO-35
- removed SPACE: KEYSWITCH-RGBLED-MX-6.25U-RGB, Keyboard:KEYSWITCH-RGBLED-MX-6.25U-RGB
Connections:
- removed net ROW1.5: DBACKSONG.C, DESC.C, DF1.C, DF10.C, DF11.C, DF12.C, DF2.C, DF3.C, DF4.C, DF5.C, DF6.C, DF7.C, DF8.C, DF9.C, DNEXTSONG.C, DPAUSE.C, DPAUSEPLAY.C, DPRTSC.C, DRANDSONG.C, DSCROLLLOCK.C, DVOLUMEUP.C, DVOLUMNEDOWN.C
- removed net ROW2.5: D0.C, D1.C, D2.C, D3.C, D4.C, D5.C, D6.C, D7.C, D8.C, D9.C, DBACKSPACE.C, DDASH.C, DEQUAL.C, DGRAVE.C, DHOME.C, DINSERT.C, DKP_ASTERISK.C, DKP_DASH.C, DKP_SLASH.C, DNUMLOCK.C, DPGUP.C, DUNDERSCORE.C
- removed net ROW3.5: DBACKSLASH.C, DDELETE.C, DE.C, DEND.C, DI.C, DKP_7.C, DKP_8.C, DKP_9.C, DLBRACKET.C, DO.C, DP.C, DPGDN.C, DQ.C, DR.C, DRBRACKET.C, DT.C, DTAB.C, DU.C, DW.C, DY.C
- removed net ROW4.5: DA.C, DCAPSLOCK.C, DD.C, DENTER.C, DF.C, DG.C, DH.C, DJ.C, DK.C, DKP_4.C, DKP_52.C, DKP_6.C, DKP_62.C, DL.C, DQUOTE.C, DS.C, DSEMICOLON.C
- removed net ROW5.5: DB.C, DC.C, DCOMMA.C, DKP_1.C, DKP_2.C, DKP_3.C, DM.C, DN.C, DPERIOD.C, DSHIFT.C, DSHIFT2.C, DSLASH.C, DUP.C, DV.C, DX.C, DZ.C
- removed net ROW6.5: DALT.C, DALT2.C, DBACKSPACE_1.C, DCTRL.C, DCTRL2.C, DDOWN.C, DKP_0.C, DKP_DEL.C, DLEFT.C, DMENU.C, DRIGHT.C, DSPACE.C, DWIN.C, DWIN2.C

Commit message: Final Revision on positioning
Parts:
- added 0, 1, 2, 3, 4, 5, 6, 7, 8, 9, A, ALT, ALT2, B, BACKSLASH, BACKSONG, BACKSPACE_1, C, CAPSLOCK, COMMA, CTRL, CTRL2, D, DASH, DELETE, DELETE2, DOWN, E, END, ENTER2, EQUAL, EQUAL2, ESC, F, F1, F10, F11, F12, F2, F3, F4, F5, F6, F7, F8, F9, G, GRAVE, H, HOME, I, INSERT, J, K, KP_1, KP_2, KP_3, KP_4, KP_5, KP_52, KP_6, KP_62, KP_7, KP_8, KP_9, KP_ASTERISK, KP_DASH, KP_DEL, KP_SLASH, L, LBRACKET, LEFT, M, MENU, N, NEXTSONG, NUMLOCK, O, P, PAUSE, PAUSEPLAY, PERIOD, PGDN, PGUP, PRTSC, Q, QUOTE, R, RANDSONG, RBRACKET, RIGHT, S, SCROLLLOCK, SEMICOLON, SLASH, T, TAB, U, UNDERSCORE, UP, V, VOLUMEUP, VOLUMNEDOWN, W, WIN, WIN2, X, Y, Z: KEYSWITCH-RGBSMDLED-ALPSMX-1U-SMDRGB, Keyboard:KEYSWITCH-RGBSMDLED-ALPSMX-1U-SMDRGB
- added BACKSPACE, ENTER, KP_0, SHIFT, SHIFT2: KEYSWITCH-RGBSMDLED-ALPSMX-2U-SMDRGB, Keyboard:KEYSWITCH-RGBSMDLED-ALPSMX-2U-SMDRGB
- added D0, D1, D2, D3, D4, D5, D6, D7, D8, D9, DA, DALT, DALT2, DB, DBACKSLASH, DBACKSONG, DBACKSPACE, DBACKSPACE_1, DC, DCAPSLOCK, DCOMMA, DCTRL, DCTRL2, DD, DDASH, DDELETE, DDELETE2, DDOWN, DE, DEND, DENTER, DENTER2, DEQUAL, DEQUAL2, DESC, DF, DF1, DF10, DF11, DF12, DF2, DF3, DF4, DF5, DF6, DF7, DF8, DF9, DG, DGRAVE, DH, DHOME, DI, DINSERT, DJ, DK, DKP_0, DKP_1, DKP_2, DKP_3, DKP_4, DKP_5, DKP_52, DKP_6, DKP_62, DKP_7, DKP_8, DKP_9, DKP_ASTERISK, DKP_DASH, DKP_DEL, DKP_SLASH, DL, DLBRACKET, DLEFT, DM, DMENU, DN, DNEXTSONG, DNUMLOCK, DO, DP, DPAUSE, DPAUSEPLAY, DPERIOD, DPGDN, DPGUP, DPRTSC, DQ, DQUOTE, DR, DRANDSONG, DRBRACKET, DRIGHT, DS, DSCROLLLOCK, DSEMICOLON, DSHIFT, DSHIFT2, DSLASH, DSPACE, DT, DTAB, DU, DUNDERSCORE, DUP, DV, DVOLUMEUP, DVOLUMNEDOWN, DW, DWIN, DWIN2, DX, DY, DZ: (no value), Components:DIODE-SOD-123
- added SPACE: KEYSWITCH-RGBSMDLED-ALPSMX-6.25U-SMDRGB, Keyboard:KEYSWITCH-RGBSMDLED-ALPSMX-6.25U-SMDRGB
Connections:
- new net N$1: DESC.A, ESC.P1
- new net N$10: DF9.A, F9.P1
- new net N$100: DENTER2.A, ENTER2.P1
- new net N$101: DDELETE2.A, DELETE2.P1
- new net N$102: CTRL.P1, DCTRL.A
- new net N$103: DWIN.A, WIN.P1
- new net N$104: ALT.P1, DALT.A
- new net N$105: DSPACE.A, SPACE.P1
- new net N$106: ALT2.P1, DALT2.A
- new net N$107: DWIN2.A, WIN2.P1
- new net N$108: DMENU.A, MENU.P1
- new net N$109: CTRL2.P1, DCTRL2.A
- new net N$11: DF10.A, F10.P1
- new net N$110: DLEFT.A, LEFT.P1
- new net N$111: DDOWN.A, DOWN.P1
- new net N$112: DRIGHT.A, RIGHT.P1
- new net N$113: DKP_0.A, KP_0.P1
- new net N$114: DKP_DEL.A, KP_DEL.P1
- new net N$115: BACKSPACE_1.P1, DBACKSPACE_1.A
- new net N$12: DF11.A, F11.P1
- new net N$13: DF12.A, F12.P1
- new net N$14: DVOLUMEUP.A, VOLUMEUP.P1
- new net N$15: DVOLUMNEDOWN.A, VOLUMNEDOWN.P1
- new net N$16: DPRTSC.A, PRTSC.P1
- new net N$17: DSCROLLLOCK.A, SCROLLLOCK.P1
- new net N$18: DPAUSE.A, PAUSE.P1
- new net N$19: BACKSONG.P1, DBACKSONG.A
- new net N$2: DF1.A, F1.P1
- new net N$20: DPAUSEPLAY.A, PAUSEPLAY.P1
- new net N$21: DNEXTSONG.A, NEXTSONG.P1
- new net N$22: DRANDSONG.A, RANDSONG.P1
- new net N$23: DGRAVE.A, GRAVE.P1
- new net N$24: 1.P1, D1.A
- new net N$25: 2.P1, D2.A
- new net N$26: 3.P1, D3.A
- new net N$27: 4.P1, D4.A
- new net N$28: 5.P1, D5.A
- new net N$29: 6.P1, D6.A
- new net N$3: DF2.A, F2.P1
- new net N$30: 7.P1, D7.A
- new net N$31: 8.P1, D8.A
- new net N$32: 9.P1, D9.A
- new net N$33: 0.P1, D0.A
- new net N$34: DASH.P1, DDASH.A
- new net N$35: DEQUAL.A, EQUAL.P1
- new net N$36: BACKSPACE.P1, DBACKSPACE.A
- new net N$37: DINSERT.A, INSERT.P1
- new net N$38: DHOME.A, HOME.P1
- new net N$39: DPGUP.A, PGUP.P1
- new net N$4: DF3.A, F3.P1
- new net N$40: DNUMLOCK.A, NUMLOCK.P1
- new net N$41: DKP_SLASH.A, KP_SLASH.P1
- new net N$42: DKP_ASTERISK.A, KP_ASTERISK.P1
- new net N$43: DKP_DASH.A, KP_DASH.P1
- new net N$44: DUNDERSCORE.A, UNDERSCORE.P1
- new net N$45: DTAB.A, TAB.P1
- new net N$46: DQ.A, Q.P1
- new net N$47: DW.A, W.P1
- new net N$48: DE.A, E.P1
- new net N$49: DR.A, R.P1
- new net N$5: DF4.A, F4.P1
- new net N$50: DT.A, T.P1
- new net N$51: DY.A, Y.P1
- new net N$52: DU.A, U.P1
- new net N$53: DI.A, I.P1
- new net N$54: DO.A, O.P1
- new net N$55: DP.A, P.P1
- new net N$56: DLBRACKET.A, LBRACKET.P1
- new net N$57: DRBRACKET.A, RBRACKET.P1
- new net N$58: BACKSLASH.P1, DBACKSLASH.A
- new net N$59: DDELETE.A, DELETE.P1
- new net N$6: DF5.A, F5.P1
- new net N$60: DEND.A, END.P1
- new net N$61: DPGDN.A, PGDN.P1
- new net N$62: DKP_7.A, KP_7.P1
- new net N$63: DKP_8.A, KP_8.P1
- new net N$64: DKP_9.A, KP_9.P1
- new net N$65: DEQUAL2.A, EQUAL2.P1
- new net N$66: DKP_5.A, KP_5.P1
- new net N$67: CAPSLOCK.P1, DCAPSLOCK.A
- new net N$68: A.P1, DA.A
- new net N$69: DS.A, S.P1
- new net N$7: DF6.A, F6.P1
- new net N$70: D.P1, DD.A
- new net N$71: DF.A, F.P1
- new net N$72: DG.A, G.P1
- new net N$73: DH.A, H.P1
- new net N$74: DJ.A, J.P1
- new net N$75: DK.A, K.P1
- new net N$76: DL.A, L.P1
- new net N$77: DSEMICOLON.A, SEMICOLON.P1
- new net N$78: DQUOTE.A, QUOTE.P1
- new net N$79: DENTER.A, ENTER.P1
- new net N$8: DF7.A, F7.P1
- new net N$80: DKP_4.A, KP_4.P1
- new net N$81: DKP_52.A, KP_52.P1
- new net N$82: DKP_6.A, KP_6.P1
- new net N$83: DKP_62.A, KP_62.P1
- new net N$84: DSHIFT.A, SHIFT.P1
- new net N$85: DZ.A, Z.P1
- new net N$86: DX.A, X.P1
- new net N$87: C.P1, DC.A
- new net N$88: DV.A, V.P1
- new net N$89: B.P1, DB.A
- new net N$9: DF8.A, F8.P1
- new net N$90: DN.A, N.P1
- new net N$91: DM.A, M.P1
- new net N$92: COMMA.P1, DCOMMA.A
- new net N$93: DPERIOD.A, PERIOD.P1
- new net N$94: DSLASH.A, SLASH.P1
- new net N$95: DSHIFT2.A, SHIFT2.P1
- new net N$96: DUP.A, UP.P1
- new net N$97: DKP_1.A, KP_1.P1
- new net N$98: DKP_2.A, KP_2.P1
- new net N$99: DKP_3.A, KP_3.P1
- new net ROW1.5: DBACKSONG.C, DESC.C, DF1.C, DF10.C, DF11.C, DF12.C, DF2.C, DF3.C, DF4.C, DF5.C, DF6.C, DF7.C, DF8.C, DF9.C, DNEXTSONG.C, DPAUSE.C, DPAUSEPLAY.C, DPRTSC.C, DRANDSONG.C, DSCROLLLOCK.C, DVOLUMEUP.C, DVOLUMNEDOWN.C
- new net ROW2.5: D0.C, D1.C, D2.C, D3.C, D4.C, D5.C, D6.C, D7.C, D8.C, D9.C, DBACKSPACE.C, DDASH.C, DEQUAL.C, DGRAVE.C, DHOME.C, DINSERT.C, DKP_ASTERISK.C, DKP_DASH.C, DKP_SLASH.C, DNUMLOCK.C, DPGUP.C, DUNDERSCORE.C
- new net ROW3.5: DBACKSLASH.C, DDELETE.C, DE.C, DEND.C, DEQUAL2.C, DI.C, DKP_5.C, DKP_7.C, DKP_8.C, DKP_9.C, DLBRACKET.C, DO.C, DP.C, DPGDN.C, DQ.C, DR.C, DRBRACKET.C, DT.C, DTAB.C, DU.C, DW.C, DY.C
- new net ROW4.5: DA.C, DCAPSLOCK.C, DD.C, DENTER.C, DF.C, DG.C, DH.C, DJ.C, DK.C, DKP_4.C, DKP_52.C, DKP_6.C, DKP_62.C, DL.C, DQUOTE.C, DS.C, DSEMICOLON.C
- new net ROW5.5: DB.C, DC.C, DCOMMA.C, DDELETE2.C, DENTER2.C, DKP_1.C, DKP_2.C, DKP_3.C, DM.C, DN.C, DPERIOD.C, DSHIFT.C, DSHIFT2.C, DSLASH.C, DUP.C, DV.C, DX.C, DZ.C
- new net ROW6.5: DALT.C, DALT2.C, DBACKSPACE_1.C, DCTRL.C, DCTRL2.C, DDOWN.C, DKP_0.C, DKP_DEL.C, DLEFT.C, DMENU.C, DRIGHT.C, DSPACE.C, DWIN.C, DWIN2.C

Commit message: Fixed Board
Parts:
- renumbered DELETE2 to KP_DELETE2
Changed lines of the file:
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@@
 <part name="ENTER2" library="Keyboard" deviceset="KEYSWITCH-RGBSMDLED" device="-ALPSMX-1U-SMDRGB"/>
 <part name="DENTER2" library="Components" deviceset="DIODE" device="-SOD-123"/>
-<part name="DELETE2" library="Keyboard" deviceset="KEYSWITCH-RGBSMDLED" device="-ALPSMX-1U-SMDRGB"/>
+<part name="KP_DELETE2" library="Keyboard" deviceset="KEYSWITCH-RGBSMDLED" device="-ALPSMX-1U-SMDRGB"/>
 <part name="DDELETE2" library="Components" deviceset="DIODE" device="-SOD-123"/>
 <part name="CTRL" library="Keyboard" deviceset="KEYSWITCH-RGBSMDLED" device="-ALPSMX-1U-SMDRGB"/>
@@
 <attribute name="VALUE" x="936.6758" y="-273.0754" size="1.778" layer="96" rot="R90"/>
 </instance>
-<instance part="DELETE2" gate="G$1" x="963.93" y="-266.7" smashed="yes">
+<instance part="KP_DELETE2" gate="G$1" x="963.93" y="-266.7" smashed="yes">
 <attribute name="NAME" x="957.12" y="-261.382" size="1" layer="95"/>
 </instance>
@@
 <net name="N$101" class="0">
 <segment>
-<pinref part="DELETE2" gate="G$1" pin="P1"/>
+<pinref part="KP_DELETE2" gate="G$1" pin="P1"/>
 <pinref part="DDELETE2" gate="D$1" pin="A"/>
 </segment>

Commit message: Updated alot and am having fun
Parts:
- added C1, C2: 22pF, rcl:C-EUC0805
- added C3, C4, C5, C6, C7: 0.1uF, rcl:C-EUC0805
- added C8: 1u, rcl:C-EUC0805
- added DLOCK, DM1, DM2, DM3, DM4, DM5, DM6: (no value), Components:DIODE-SOD-123
- added J1: (no value), SparkFun-Connectors:USB_MICRO-B_FEMALE-SMT
- added LOCK, M6: KEYSWITCH-RGBSMDLED-ALPSMX-1U-SMDRGB, Keyboard:KEYSWITCH-RGBSMDLED-ALPSMX-1U-SMDRGB
- added M1, M2, M3, M4, M5: KEYSWITCH-RGBSMDLED-MX-1U-SMDRGB, Keyboard:KEYSWITCH-RGBSMDLED-MX-1U-SMDRGB
- added R1, R2: 10k, rcl:R-US_M0805
- added R3, R4: 22, rcl:R-US_M0805
- added S1: (no value), switch-omron:31-XX
- added U$1: 32U4, SparkFun-IC-Microcontroller:ATMEGA32U4TQFP-44
- added Y1: (no value), SparkFun-Clocks:CRYSTALSMD-3.2X2.5
- renumbered DRANDSONG to DNEXTSONG1
Connections:
- removed net ROW1.5: DBACKSONG.C, DESC.C, DF1.C, DF10.C, DF11.C, DF12.C, DF2.C, DF3.C, DF4.C, DF5.C, DF6.C, DF7.C, DF8.C, DF9.C, DNEXTSONG.C, DNEXTSONG1.C, DPAUSE.C, DPAUSEPLAY.C, DPRTSC.C, DSCROLLLOCK.C, DVOLUMEUP.C, DVOLUMNEDOWN.C
- removed net ROW2.5: D0.C, D1.C, D2.C, D3.C, D4.C, D5.C, D6.C, D7.C, D8.C, D9.C, DBACKSPACE.C, DDASH.C, DEQUAL.C, DGRAVE.C, DHOME.C, DINSERT.C, DKP_ASTERISK.C, DKP_DASH.C, DKP_SLASH.C, DNUMLOCK.C, DPGUP.C, DUNDERSCORE.C
- removed net ROW3.5: DBACKSLASH.C, DDELETE.C, DE.C, DEND.C, DEQUAL2.C, DI.C, DKP_5.C, DKP_7.C, DKP_8.C, DKP_9.C, DLBRACKET.C, DO.C, DP.C, DPGDN.C, DQ.C, DR.C, DRBRACKET.C, DT.C, DTAB.C, DU.C, DW.C, DY.C
- removed net ROW4.5: DA.C, DCAPSLOCK.C, DD.C, DENTER.C, DF.C, DG.C, DH.C, DJ.C, DK.C, DKP_4.C, DKP_52.C, DKP_6.C, DKP_62.C, DL.C, DQUOTE.C, DS.C, DSEMICOLON.C
- removed net ROW5.5: DB.C, DC.C, DCOMMA.C, DDELETE2.C, DENTER2.C, DKP_1.C, DKP_2.C, DKP_3.C, DM.C, DN.C, DPERIOD.C, DSHIFT.C, DSHIFT2.C, DSLASH.C, DUP.C, DV.C, DX.C, DZ.C
- removed net ROW6.5: DALT.C, DALT2.C, DBACKSPACE_1.C, DCTRL.C, DCTRL2.C, DDOWN.C, DKP_0.C, DKP_DEL.C, DLEFT.C, DMENU.C, DRIGHT.C, DSPACE.C, DWIN.C, DWIN2.C
- new net +5V: C3.1, C4.1, C5.1, C6.1, C7.1, J1.VBUS, R1.1, U$1.AVCC@24, U$1.AVCC@44, U$1.UVCC, U$1.VCC@14, U$1.VCC@34
- new net GND: C1.2, C2.2, C3.2, C4.2, C5.2, C6.2, C7.2, C8.1, J1.GND, J1.SHIELD, R2.1, S1.P, U$1.GND@15, U$1.GND@23, U$1.GND@35, U$1.GND@43, U$1.UGND
- new net N$116: C1.1, U$1.XTAL1, Y1.1
- new net N$117: C2.1, U$1.XTAL2, Y1.2
- new net N$118: R1.2, S1.S, U$1.!RESET
- new net N$119: R2.2, U$1.PE2/!HWB
- new net N$120: DM6.A, M6.P1
- new net N$121: J1.D+, R3.1
- new net N$122: J1.D-, R4.1
- new net N$123: R3.2, U$1.D+
- new net N$124: R4.2, U$1.D-
- new net N$125: C8.2, U$1.UCAP
- new net N$126: DM1.A, M1.P1
- new net N$127: DM2.A, M2.P1
- new net N$128: DM3.A, M3.P1
- new net N$129: DM4.A, M4.P1
- new net N$130: DM5.A, M5.P1
- new net N$132: DF1.C, DF11.C, DF3.C, DF5.C, DF7.C, DF9.C, DM6.C, DNEXTSONG1.C, DPAUSE.C, DPAUSEPLAY.C, DPRTSC.C, DVOLUMEUP.C
- new net N$133: DBACKSONG.C, DESC.C, DF10.C, DF12.C, DF2.C, DF4.C, DF6.C, DF8.C, DLOCK.C, DNEXTSONG.C, DSCROLLLOCK.C, DVOLUMNEDOWN.C
- new net N$134: D1.C, D3.C, D5.C, D7.C, D9.C, DDASH.C, DINSERT.C, DKP_DASH.C, DKP_SLASH.C, DM5.C, DPGUP.C
- new net N$135: D0.C, D2.C, D4.C, D6.C, D8.C, DBACKSPACE.C, DEQUAL.C, DGRAVE.C, DHOME.C, DKP_ASTERISK.C, DNUMLOCK.C, DUNDERSCORE.C
- new net N$139: A.P0
- new net N$140: MENU.P0
- new net N$153: J.P0
- new net N$154: KP_DELETE2.P0
- new net N$22: DLOCK.A, LOCK.P1
Other:
- moved on the sheet: DENTER, DF11, DVOLUMNEDOWN, ENTER, F11

Commit message: Updated Schematic
Parts:
- removed M2, M3, M4, M5: KEYSWITCH-RGBSMDLED-MX-1U-SMDRGB, Keyboard:KEYSWITCH-RGBSMDLED-MX-1U-SMDRGB
- removed Y1: (no value), SparkFun-Clocks:CRYSTALSMD-3.2X2.5
- added CAPSLOCK1, GRAVE1, TAB1: KEYSWITCH-RGBSMDLED-ALPSMX-1U-SMDRGB, Keyboard:KEYSWITCH-RGBSMDLED-ALPSMX-1U-SMDRGB
- added SHIFT1: KEYSWITCH-RGBSMDLED-ALPSMX-2U-SMDRGB, Keyboard:KEYSWITCH-RGBSMDLED-ALPSMX-2U-SMDRGB
- added Y2: CRYSTAL-GROUNDEDSMD-3.2X2.5, SparkFun-Clocks:CRYSTAL-GROUNDEDSMD-3.2X2.5
- renumbered M6 to ESC1
Connections:
- net +5V renamed VCC
- removed net N$126: DM1.A, M1.P1
- removed net N$132: DF1.C, DF11.C, DF3.C, DF5.C, DF7.C, DF9.C, DM6.C, DNEXTSONG1.C, DPAUSE.C, DPAUSEPLAY.C, DPRTSC.C, DVOLUMEUP.C
- removed net N$133: DBACKSONG.C, DESC.C, DF10.C, DF12.C, DF2.C, DF4.C, DF6.C, DF8.C, DLOCK.C, DNEXTSONG.C, DSCROLLLOCK.C, DVOLUMNEDOWN.C
- removed net N$134: D1.C, D3.C, D5.C, D7.C, D9.C, DDASH.C, DINSERT.C, DKP_DASH.C, DKP_SLASH.C, DM5.C, DPGUP.C
- removed net N$135: D0.C, D2.C, D4.C, D6.C, D8.C, DBACKSPACE.C, DEQUAL.C, DGRAVE.C, DHOME.C, DKP_ASTERISK.C, DNUMLOCK.C, DUNDERSCORE.C
- removed net N$139: A.P0
- removed net N$140: MENU.P0
- removed net N$153: J.P0
- removed net N$154: KP_DELETE2.P0
- new net COL1: CAPSLOCK.P0, CAPSLOCK1.P0, ESC.P0, ESC1.P0, GRAVE.P0, GRAVE1.P0, M1.P0, SHIFT.P0, SHIFT1.P0, TAB.P0, TAB1.P0, U$1.PF7(ADC7)
- new net COL10: BACKSONG.P0, ENTER2.P0, KP_3.P0, KP_6.P0, KP_7.P0, KP_8.P0, KP_DEL.P0, KP_SLASH.P0, NUMLOCK.P0, PAUSE.P0, U$1.PC6
- new net COL11: EQUAL2.P0, KP_9.P0, KP_ASTERISK.P0, KP_DASH.P0, NEXTSONG.P0, PAUSEPLAY.P0, U$1.PD7(ADC10)
- new net COL12: BACKSPACE_1.P0, KP_5.P0, KP_62.P0, KP_DELETE2.P0, LOCK.P0, RANDSONG.P0, U$1.PE6, UNDERSCORE.P0
- new net COL2: 1.P0, 2.P0, A.P0, CTRL.P0, F1.P0, F2.P0, Q.P0, S.P0, U$1.PF6(ADC6), W.P0, X.P0, Z.P0
- new net COL3: 3.P0, 4.P0, C.P0, D.P0, E.P0, F.P0, F3.P0, F4.P0, R.P0, U$1.PF5(ADC5), V.P0, WIN.P0
- new net COL4: 5.P0, 6.P0, ALT.P0, B.P0, F5.P0, F6.P0, G.P0, H.P0, N.P0, T.P0, U$1.PF4(ADC4), Y.P0
- new net COL5: 7.P0, 8.P0, COMMA.P0, F7.P0, F8.P0, I.P0, J.P0, K.P0, M.P0, SPACE.P0, U$1.PF1(ADC1), U.P0
- new net COL6: 0.P0, 9.P0, ALT2.P0, F10.P0, F9.P0, L.P0, O.P0, P.P0, PERIOD.P0, SEMICOLON.P0, SLASH.P0, U$1.PF0(ADC0)
- new net COL7: DASH.P0, ENTER.P0, EQUAL.P0, F11.P0, F12.P0, LBRACKET.P0, MENU.P0, QUOTE.P0, RBRACKET.P0, SHIFT2.P0, U$1.PD1(SDA), WIN2.P0
- new net COL8: BACKSLASH.P0, BACKSPACE.P0, CTRL2.P0, DELETE.P0, DOWN.P0, INSERT.P0, LEFT.P0, RIGHT.P0, U$1.PD0(SCL), UP.P0, VOLUMEUP.P0, VOLUMNEDOWN.P0
- new net COL9: END.P0, HOME.P0, KP_0.P0, KP_1.P0, KP_2.P0, KP_4.P0, KP_52.P0, PGDN.P0, PGUP.P0, PRTSC.P0, SCROLLLOCK.P0, U$1.PD4(ADC8)
- new net ROW1.1: DF1.C, DF11.C, DF3.C, DF5.C, DF7.C, DF9.C, DM6.C, DNEXTSONG1.C, DPAUSE.C, DPAUSEPLAY.C, DSCROLLLOCK.C, DVOLUMEUP.C, U$1.PB4(ADC11)
- new net ROW1.2: DBACKSONG.C, DESC.C, DF10.C, DF12.C, DF2.C, DF4.C, DF6.C, DF8.C, DLOCK.C, DNEXTSONG.C, DPRTSC.C, DVOLUMNEDOWN.C, U$1.PB5(ADC12)
- new net ROW2.1: D1.C, D3.C, D5.C, D7.C, D9.C, DBACKSPACE.C, DDASH.C, DHOME.C, DKP_DASH.C, DKP_SLASH.C, DM5.C, U$1.PB6(ADC13)
- new net ROW2.2: D0.C, D2.C, D4.C, D6.C, D8.C, DEQUAL.C, DGRAVE.C, DINSERT.C, DKP_ASTERISK.C, DNUMLOCK.C, DPGUP.C, DUNDERSCORE.C, U$1.PB7
- new net ROW3.1: DBACKSLASH.C, DE.C, DEND.C, DEQUAL2.C, DKP_8.C, DLBRACKET.C, DM4.C, DO.C, DQ.C, DT.C, DU.C, U$1.PD6(ADC9)
- new net ROW3.2: DDELETE.C, DI.C, DKP_5.C, DKP_7.C, DKP_9.C, DP.C, DPGDN.C, DR.C, DRBRACKET.C, DTAB.C, DW.C, DY.C, U$1.PC7
- new net ROW4.1: DA.C, DCTRL2.C, DD.C, DG.C, DJ.C, DKP_4.C, DKP_6.C, DKP_62.C, DL.C, DM3.C, DQUOTE.C, U$1.PB0(SS)
- new net ROW4.2: DCAPSLOCK.C, DENTER.C, DENTER2.C, DF.C, DH.C, DK.C, DKP_52.C, DS.C, DSEMICOLON.C, DUP.C, U$1.PB1(SCK)
- new net ROW5.1: DB.C, DC.C, DKP_2.C, DLEFT.C, DM.C, DM2.C, DMENU.C, DPERIOD.C, DZ.C, U$1.PB2(MOSI)
- new net ROW5.2: DCOMMA.C, DDELETE2.C, DKP_1.C, DKP_3.C, DN.C, DRIGHT.C, DSHIFT.C, DSHIFT2.C, DSLASH.C, DV.C, DX.C, U$1.PB3(MISO)
- new net ROW6.1: DALT.C, DALT2.C, DBACKSPACE_1.C, DCTRL.C, DDOWN.C, DKP_0.C, DKP_DEL.C, DM1.C, DSPACE.C, DWIN.C, DWIN2.C, U$1.PD5
- net GND: now also Y2.3
- net N$116: now also Y2.1; no longer Y1.1
- net N$117: now also Y2.2; no longer Y1.2
- net N$127: now also DM5.A, GRAVE1.P1; no longer DM2.A, M2.P1
- net N$128: now also DM4.A, TAB1.P1; no longer DM3.A, M3.P1
- net N$129: now also CAPSLOCK1.P1, DM3.A; no longer DM4.A, M4.P1
- net N$130: now also DM2.A, SHIFT1.P1; no longer DM5.A, M5.P1
Other:
- moved on the sheet: 2, D2
