File: Keyboard_PCB/keyboard_schematic.sch (EAGLE design)
At the start: 262 parts, among them J1 1-2295018-2, M2 KEYSWITCH-RGBSMDLED-ALPSMX-1U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, M3 KEYSWITCH-RGBSMDLED-ALPSMX-1U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, M4 KEYSWITCH-RGBSMDLED-ALPSMX-1U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, M5 KEYSWITCH-RGBSMDLED-ALPSMX-1U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, M6 KEYSWITCH-RGBSMDLED-ALPSMX-1U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, Y2 CRYSTAL-GROUNDEDSMD-3.2X2.5

Commit message: Updated Board
Parts:
- removed EQUAL2: KEYSWITCH-RGBSMDLED-ALPSMX-1U-SMDRGB, Keyboard:KEYSWITCH-RGBSMDLED-ALPSMX-1U-SMDRGB
- added PLUS2: KEYSWITCH-RGBSMDLED-ALPSMX-2U-SMDRGB-ROTATED, Keyboard:KEYSWITCH-RGBSMDLED-ALPSMX-2U-SMDRGB-ROTATED
- ENTER2: value KEYSWITCH-RGBSMDLED-ALPSMX-1U-SMDRGB -> KEYSWITCH-RGBSMDLED-ALPSMX-2U-SMDRGB-ROTATED; device Keyboard:KEYSWITCH-RGBSMDLED-ALPSMX-1U-SMDRGB -> Keyboard:KEYSWITCH-RGBSMDLED-ALPSMX-2U-SMDRGB-ROTATED
Connections:
- net COL24: now also PLUS2.P0; no longer EQUAL2.P0
- net N$193: now also PLUS2.DI; no longer EQUAL2.DI
- net N$194: now also PLUS2.DO; no longer EQUAL2.DO
- net N$65: now also PLUS2.P1; no longer EQUAL2.P1
Changed lines of the file:
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@@
 <part name="KP_9" library="Keyboard" deviceset="KEYSWITCH-RGBSMDLED" device="-ALPSMX-1U-SMDRGB"/>
 <part name="DKP_9" library="Components" deviceset="DIODE" device="-SOD-123"/>
-<part name="EQUAL2" library="Keyboard" deviceset="KEYSWITCH-RGBSMDLED" device="-ALPSMX-1U-SMDRGB"/>
 <part name="DEQUAL2" library="Components" deviceset="DIODE" device="-SOD-123"/>
 <part name="KP_5" library="Keyboard" deviceset="KEYSWITCH-RGBSMDLED" device="-ALPSMX-1U-SMDRGB"/>
@@
 <part name="KP_3" library="Keyboard" deviceset="KEYSWITCH-RGBSMDLED" device="-ALPSMX-1U-SMDRGB"/>
 <part name="DKP_3" library="Components" deviceset="DIODE" device="-SOD-123"/>
-<part name="ENTER2" library="Keyboard" deviceset="KEYSWITCH-RGBSMDLED" device="-ALPSMX-1U-SMDRGB"/>
 <part name="DENTER2" library="Components" deviceset="DIODE" device="-SOD-123"/>
 <part name="KP_DELETE2" library="Keyboard" deviceset="KEYSWITCH-RGBSMDLED" device="-ALPSMX-1U-SMDRGB"/>
@@
 <part name="P+11" library="supply1" library_urn="urn:adsk.eagle:library:371" deviceset="+5V" device=""/>
 <part name="C7" library="rcl" library_urn="urn:adsk.eagle:library:334" deviceset="C-EU" device="C0805" package3d_urn="urn:adsk.eagle:package:23617/2" value="0.1uF"/>
+<part name="PLUS2" library="Keyboard" deviceset="KEYSWITCH-RGBSMDLED" device="-ALPSMX-2U-SMDRGB-ROTATED"/>
+<part name="ENTER2" library="Keyboard" deviceset="KEYSWITCH-RGBSMDLED" device="-ALPSMX-2U-SMDRGB-ROTATED"/>
 </parts>
 <sheets>
@@
 <attribute name="VALUE" x="897.3058" y="-121.9454" size="1.778" layer="96" rot="R90"/>
 </instance>
-<instance part="EQUAL2" gate="G$1" x="929.64" y="-134.62" smashed="yes">
-<attribute name="NAME" x="922.83" y="-129.302" size="1" layer="95"/>
-</instance>
 <instance part="DEQUAL2" gate="D$1" x="929.64" y="-119.38" smashed="yes" rot="R90">
 <attribute name="NAME" x="926.9984" y="-121.6914" size="1.778" layer="95" rot="R90"/>
@@
 <attribute name="VALUE" x="897.3058" y="-254.0254" size="1.778" layer="96" rot="R90"/>
 </instance>
-<instance part="ENTER2" gate="G$1" x="929.64" y="-266.7" smashed="yes">
-<attribute name="NAME" x="922.83" y="-261.382" size="1" layer="95"/>
-</instance>
 <instance part="DENTER2" gate="D$1" x="929.64" y="-251.46" smashed="yes" rot="R90">
 <attribute name="NAME" x="926.9984" y="-253.7714" size="1.778" layer="95" rot="R90"/>
@@
 <attribute name="NAME" x="550.593" y="-190.262" size="1" layer="95"/>
 </instance>
+<instance part="PLUS2" gate="G$1" x="929.64" y="-134.62" smashed="yes">
+<attribute name="NAME" x="922.83" y="-129.302" size="1" layer="95"/>
+</instance>
+<instance part="ENTER2" gate="G$1" x="929.64" y="-266.7" smashed="yes">
+<attribute name="NAME" x="922.83" y="-261.382" size="1" layer="95"/>
+</instance>
 </instances>
 <busses>
@@
 </segment>
 </net>
-<net name="N$65" class="0">
-<segment>
-<pinref part="EQUAL2" gate="G$1" pin="P1"/>
-<pinref part="DEQUAL2" gate="D$1" pin="A"/>
-</segment>
-</net>
 <net name="N$66" class="0">
 <segment>
@@
 </segment>
 </net>
-<net name="N$100" class="0">
-<segment>
-<pinref part="ENTER2" gate="G$1" pin="P1"/>
-<pinref part="DENTER2" gate="D$1" pin="A"/>
-</segment>
-</net>
 <net name="N$101" class="0">
 <segment>
@@
 <segment>
 <pinref part="RANDSONG" gate="G$1" pin="P0"/>
-<pinref part="ENTER2" gate="G$1" pin="P0"/>
 <wire x1="919.48" y1="2.54" x2="919.48" y2="-63.5" width="0.1524" layer="91"/>
 <pinref part="KP_DASH" gate="G$1" pin="P0"/>
-<wire x1="919.48" y1="-63.5" x2="919.48" y2="-132.08" width="0.1524" layer="91"/>
 <junction x="919.48" y="-63.5"/>
-<pinref part="EQUAL2" gate="G$1" pin="P0"/>
+<wire x1="919.48" y1="-63.5" x2="919.48" y2="-132.08" width="0.1524" layer="91"/>
+<label x="922.02" y="-33.02" size="1.778" layer="95"/>
+<pinref part="PLUS2" gate="G$1" pin="P0"/>
 <wire x1="919.48" y1="-132.08" x2="919.48" y2="-264.16" width="0.1524" layer="91"/>
 <junction x="919.48" y="-132.08"/>
-<label x="922.02" y="-33.02" size="1.778" layer="95"/>
+<pinref part="ENTER2" gate="G$1" pin="P0"/>
 </segment>
 </net>
@@
 <wire x1="924.56" y1="-149.86" x2="924.56" y2="-144.78" width="0.1524" layer="91"/>
 <pinref part="KP_9" gate="G$1" pin="DO"/>
-<pinref part="EQUAL2" gate="G$1" pin="DI"/>
+<pinref part="PLUS2" gate="G$1" pin="DI"/>
 </segment>
 </net>
@@
 <wire x1="927.1" y1="-149.86" x2="958.85" y2="-149.86" width="0.1524" layer="91"/>
 <wire x1="958.85" y1="-149.86" x2="958.85" y2="-144.78" width="0.1524" layer="91"/>
-<pinref part="EQUAL2" gate="G$1" pin="DO"/>
 <pinref part="KP_5" gate="G$1" pin="DI"/>
+<pinref part="PLUS2" gate="G$1" pin="DO"/>
 </segment>
 </net>
@@
 <pinref part="KP_3" gate="G$1" pin="DO"/>
 <wire x1="890.27" y1="-276.86" x2="890.27" y2="-281.94" width="0.1524" layer="91"/>
-<pinref part="ENTER2" gate="G$1" pin="DI"/>
 <wire x1="890.27" y1="-281.94" x2="924.56" y2="-281.94" width="0.1524" layer="91"/>
 <wire x1="924.56" y1="-281.94" x2="924.56" y2="-276.86" width="0.1524" layer="91"/>
+<pinref part="ENTER2" gate="G$1" pin="DI"/>
 </segment>
 </net>
 <net name="N$229" class="0">
 <segment>
-<pinref part="ENTER2" gate="G$1" pin="DO"/>
 <wire x1="927.1" y1="-276.86" x2="927.1" y2="-281.94" width="0.1524" layer="91"/>
 <wire x1="927.1" y1="-281.94" x2="958.85" y2="-281.94" width="0.1524" layer="91"/>
 <pinref part="KP_DELETE2" gate="G$1" pin="DI"/>
 <wire x1="958.85" y1="-281.94" x2="958.85" y2="-276.86" width="0.1524" layer="91"/>
+<pinref part="ENTER2" gate="G$1" pin="DO"/>
 </segment>
 </net>
@@
 </segment>
 </net>
+<net name="N$65" class="0">
+<segment>
+<pinref part="DEQUAL2" gate="D$1" pin="A"/>
+<pinref part="PLUS2" gate="G$1" pin="P1"/>
+</segment>
+</net>
+<net name="N$100" class="0">
+<segment>
+<pinref part="DENTER2" gate="D$1" pin="A"/>
+<pinref part="ENTER2" gate="G$1" pin="P1"/>
+</segment>
+</net>

Commit message: Updated Board
Connections:
- net D+USB: now also J1.D+@1
- net D-USB: now also J1.D-@1
Changed lines of the file:
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@@
 <sheets>
 <sheet>
+<description>Key connections</description>
 <plain>
 </plain>
@@
 </sheet>
 <sheet>
-<description>Main Board</description>
+<description>Controller Board</description>
 <plain>
 </plain>
@@
 <pinref part="J1" gate="G$1" pin="D+"/>
 <wire x1="-162.56" y1="71.12" x2="-137.16" y2="71.12" width="0.1524" layer="91"/>
+<pinref part="J1" gate="G$1" pin="D+@1"/>
+<wire x1="-193.04" y1="71.12" x2="-162.56" y2="71.12" width="0.1524" layer="91"/>
+<junction x="-162.56" y="71.12"/>
 </segment>
 </net>
@@
 <pinref part="J1" gate="G$1" pin="D-"/>
 <wire x1="-162.56" y1="68.58" x2="-139.7" y2="68.58" width="0.1524" layer="91"/>
+<pinref part="J1" gate="G$1" pin="D-@1"/>
+<wire x1="-162.56" y1="68.58" x2="-193.04" y2="68.58" width="0.1524" layer="91"/>
+<junction x="-162.56" y="68.58"/>
 </segment>
 </net>
