File: Keyboard_PCB/keyboard_schematic.brd (EAGLE design)
At the start: 485.1 x 152.3 mm, 262 parts, among them J1 1-2295018-2, M2 KEYSWITCH-RGBSMDLED-ALPSMX-1U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, M3 KEYSWITCH-RGBSMDLED-ALPSMX-1U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, M4 KEYSWITCH-RGBSMDLED-ALPSMX-1U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, M5 KEYSWITCH-RGBSMDLED-ALPSMX-1U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, M6 KEYSWITCH-RGBSMDLED-ALPSMX-1U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, Y2 CRYSTAL-GROUNDEDSMD-3.2X2.5

Commit message: Updated Board
Parts:
- moved R3 0.51 mm to (431.3, 136.7)
- moved R4 0.51 mm to (431.3, 134.6)
Connections:
- net D+USB: now also J1.B6
- net D-USB: now also J1.B7
Routing:
- net D-USB: track 4.22 -> 11.8 mm, vias 0 -> 2
- net XTAL2: track 12.0 -> 7.93 mm
- net D+USB: track 2.87 -> 4.89 mm
- net D+32U: track 15.0 -> 14.5 mm
- net D-32U4: track 19.4 -> 18.9 mm
