File: Keyboard_PCB/keyboard.brd (EAGLE design)
At the start: 487.7 x 175.3 mm, 262 parts, among them J1 1-2295018-2, M2 KEYSWITCH-RGBSMDLED-ALPSMX-1U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, M3 KEYSWITCH-RGBSMDLED-ALPSMX-1U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, M4 KEYSWITCH-RGBSMDLED-ALPSMX-1U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, M5 KEYSWITCH-RGBSMDLED-ALPSMX-1U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, M6 KEYSWITCH-RGBSMDLED-ALPSMX-1U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, Y2 CRYSTAL-GROUNDEDSMD-3.2X2.5

Commit message: Thing
Parts:
- removed EQUAL2: KEYSWITCH-RGBSMDLED-ALPSMX-1U-SMDRGB, Keyboard:ALPSMX-1U-SMDRGB
- added PLUS2: KEYSWITCH-RGBSMDLED-ALPSMX-2U-SMDRGB-ROTATED, Keyboard:ALPSMX-2U-SMDRGB-ROTATED
- ENTER2: value KEYSWITCH-RGBSMDLED-ALPSMX-1U-SMDRGB -> KEYSWITCH-RGBSMDLED-ALPSMX-2U-SMDRGB-ROTATED; device Keyboard:ALPSMX-1U-SMDRGB -> Keyboard:ALPSMX-2U-SMDRGB-ROTATED
- moved DEQUAL2 9.48 mm to (425.5, 74.6)
- moved DENTER2 9.45 mm to (425.2, 36.5)
- moved R6 5.18 mm to (436.3, 144.3)
- moved C3 0.51 mm to (416.8, 141.5)
- moved R3 0.51 mm to (431.3, 136.7)
- moved R4 0.51 mm to (431.3, 134.6)
- moved ENTER2 0.10 mm to (416.1, 20.3)
- moved R5 0.06 mm to (432.0, 139.7)
Connections:
- removed net COL1: CTRL1.ALPS1, CTRL1.MX1, M2.ALPS1, M2.MX1, M3.ALPS1, M3.MX1, M4.ALPS1, M4.MX1, M5.ALPS1, M5.MX1, M6.ALPS1, M6.MX1
- removed net N$163: BACKSPACE.R-, EQUAL.DOUT
- removed net N$239: J1.A9
- new net COL11: 8.ALPS1, 8.MX1, COMMA.ALPS1, COMMA.MX1, F8.ALPS1, F8.MX1, I.ALPS1, I.MX1, IC3.40, K.ALPS1, K.MX1
- new net N$102: CTRL.ALPS2, CTRL.MX2, DCTRL.A
- new net N$116: BACKSPACE.DIN, EQUAL.DOUT
- net +5V: now also 0.VDD, 1.VDD, 2.VDD, 3.VDD, 4.VDD, 5.VDD, 6.VDD, 7.VDD, 8.VDD, 9.VDD, A.VDD, ALT.VDD, ALT2.VDD, B.VDD, BACKSONG.VDD, BACKSPACE_1.VDD, C.VDD, CAPSLOCK.VDD, COMMA.VDD, CTRL.VDD, CTRL1.VDD, D.VDD, DASH.VDD, DELETE.VDD, DOWN.VDD, E.VDD, END.VDD, ENTER2.VDD, EQUAL.VDD, ESC.VDD, F.VDD, F1.VDD, F10.VDD, F11.VDD, F12.VDD, F2.VDD, F3.VDD, F4.VDD, F5.VDD, F6.VDD, F7.VDD, F9.VDD, G.VDD, GRAVE.VDD, H.VDD, HOME.VDD, I.VDD, INSERT.VDD, J.VDD, J1.A9, K.VDD, KP_0.VDD, KP_1.VDD, KP_3.VDD, KP_4.VDD, KP_5.VDD, KP_6.VDD, KP_62.VDD, KP_7.VDD, KP_9.VDD, KP_ASTERISK.VDD, KP_DASH.VDD, KP_DEL.VDD, KP_DELETE2.VDD, L.VDD, LBRACKET.VDD, LEFT.VDD, LOCK.VDD, M.VDD, M2.VDD, M3.VDD, M4.VDD, M5.VDD, M6.VDD, MENU.VDD, N.VDD, NEXTSONG.VDD, NUMLOCK.VDD, O.VDD, P.VDD, PAUSE.VDD, PAUSEPLAY.VDD, PERIOD.VDD, PGDN.VDD, PGUP.VDD, PLUS2.VDD, PRTSC.VDD, Q.VDD, QUOTE.VDD, R.VDD, RANDSONG.VDD, RBRACKET.VDD, RIGHT.VDD, S.VDD, SCROLLLOCK.VDD, SEMICOLON.VDD, SHIFT.VDD, SLASH.VDD, SPACE.LED+, T.VDD, TAB.VDD, U.VDD, UNDERSCORE.VDD, UP.VDD, V.VDD, VOLUMEUP.VDD, W.VDD, WIN.VDD, WIN2.VDD, X.VDD, Y.VDD, Z.VDD
- net COL10: now also 7.ALPS1, 7.MX1, F7.ALPS1, F7.MX1, IC3.41, J.ALPS1, J.MX1, M.ALPS1, M.MX1, U.ALPS1, U.MX1; no longer 8.ALPS1, 8.MX1, COMMA.ALPS1, COMMA.MX1, F8.ALPS1, F8.MX1, I.ALPS1, I.MX1, K.ALPS1, K.MX1
- net COL12: now also IC3.39
- net COL13: now also IC3.38
- net COL14: now also IC3.37
- net COL15: now also IC3.36
- net COL16: now also IC3.35
- net COL17: now also IC3.34
- net COL18: now also IC3.33
- net COL19: now also IC3.32
- net COL2: now also CTRL1.ALPS1, CTRL1.MX1, IC3.50, M2.ALPS1, M2.MX1, M3.ALPS1, M3.MX1, M4.ALPS1, M4.MX1, M5.ALPS1, M5.MX1, M6.ALPS1, M6.MX1; no longer CAPSLOCK.ALPS1, CAPSLOCK.MX1, CTRL.ALPS1, CTRL.MX1, ESC.ALPS1, ESC.MX1, GRAVE.ALPS1, GRAVE.MX1, SHIFT.ALPS1, SHIFT.MX1, TAB.ALPS1, TAB.MX1
- net COL20: now also IC3.31
- net COL21: now also IC3.30
- net COL22: now also IC3.29
- net COL23: now also IC3.28
- net COL24: now also IC3.27, PLUS2.ALPS1, PLUS2.MX1; no longer EQUAL2.ALPS1, EQUAL2.MX1
- net COL25: now also IC3.26
- net COL3: now also CAPSLOCK.ALPS1, CAPSLOCK.MX1, CTRL.ALPS1, CTRL.MX1, ESC.ALPS1, ESC.MX1, GRAVE.ALPS1, GRAVE.MX1, IC3.49, SHIFT.ALPS1, SHIFT.MX1, TAB.ALPS1, TAB.MX1; no longer 1.ALPS1, 1.MX1, A.ALPS1, A.MX1, F1.ALPS1, F1.MX1, Q.ALPS1, Q.MX1, WIN.ALPS1, WIN.MX1, Z.ALPS1, Z.MX1
- net COL4: now also 1.ALPS1, 1.MX1, A.ALPS1, A.MX1, F1.ALPS1, F1.MX1, IC3.48, Q.ALPS1, Q.MX1, WIN.ALPS1, WIN.MX1, Z.ALPS1, Z.MX1; no longer 2.ALPS1, 2.MX1, ALT.ALPS1, ALT.MX1, F2.ALPS1, F2.MX1, S.ALPS1, S.MX1, W.ALPS1, W.MX1, X.ALPS1, X.MX1
- net COL5: now also 2.ALPS1, 2.MX1, ALT.ALPS1, ALT.MX1, F2.ALPS1, F2.MX1, IC3.47, S.ALPS1, S.MX1, W.ALPS1, W.MX1, X.ALPS1, X.MX1; no longer 3.ALPS1, 3.MX1, C.ALPS1, C.MX1, D.ALPS1, D.MX1, E.ALPS1, E.MX1, F3.ALPS1, F3.MX1
- net COL6: now also 3.ALPS1, 3.MX1, C.ALPS1, C.MX1, D.ALPS1, D.MX1, E.ALPS1, E.MX1, F3.ALPS1, F3.MX1, IC3.46; no longer 4.ALPS1, 4.MX1, F.ALPS1, F.MX1, F4.ALPS1, F4.MX1, R.ALPS1, R.MX1, V.ALPS1, V.MX1
- net COL7: now also 4.ALPS1, 4.MX1, F.ALPS1, F.MX1, F4.ALPS1, F4.MX1, IC3.45, R.ALPS1, R.MX1, V.ALPS1, V.MX1; no longer 5.ALPS1, 5.MX1, B.ALPS1, B.MX1, F5.ALPS1, F5.MX1, G.ALPS1, G.MX1, SPACE.ALPS1, SPACE.MX1, T.ALPS1, T.MX1
- net COL8: now also 5.ALPS1, 5.MX1, B.ALPS1, B.MX1, F5.ALPS1, F5.MX1, G.ALPS1, G.MX1, IC3.44, SPACE.ALPS1, SPACE.MX1, T.ALPS1, T.MX1; no longer 6.ALPS1, 6.MX1, F6.ALPS1, F6.MX1, H.ALPS1, H.MX1, N.ALPS1, N.MX1, Y.ALPS1, Y.MX1
- net COL9: now also 6.ALPS1, 6.MX1, F6.ALPS1, F6.MX1, H.ALPS1, H.MX1, IC3.42, N.ALPS1, N.MX1, Y.ALPS1, Y.MX1; no longer 7.ALPS1, 7.MX1, F7.ALPS1, F7.MX1, J.ALPS1, J.MX1, M.ALPS1, M.MX1, U.ALPS1, U.MX1
- net D+USB: now also J1.B6
- net D-USB: now also J1.B7
- net GND: now also 0.VSS, 1.VSS, 2.VSS, 3.VSS, 4.VSS, 5.VSS, 6.VSS, 7.VSS, 8.VSS, 9.VSS, A.VSS, ALT.VSS, ALT2.VSS, B.VSS, BACKSLASH.VSS, BACKSONG.VSS, BACKSPACE.VSS, BACKSPACE_1.VSS, C.VSS, CAPSLOCK.VSS, COMMA.VSS, CTRL.VSS, CTRL1.VSS, CTRL2.VSS, D.VSS, DASH.VSS, DELETE.VSS, DOWN.VSS, E.VSS, END.VSS, ENTER.VSS, ENTER2.VSS, EQUAL.VSS, ESC.VSS, F.VSS, F1.VSS, F10.VSS, F11.VSS, F12.VSS, F2.VSS, F3.VSS, F4.VSS, F5.VSS, F6.VSS, F7.VSS, F8.VSS, F9.VSS, G.VSS, GRAVE.VSS, H.VSS, HOME.VSS, I.VSS, INSERT.VSS, J.VSS, K.VSS, KP_0.VSS, KP_1.VSS, KP_2.VSS, KP_3.VSS, KP_4.VSS, KP_5.VSS, KP_52.VSS, KP_6.VSS, KP_62.VSS, KP_7.VSS, KP_8.VSS, KP_9.VSS, KP_ASTERISK.VSS, KP_DASH.VSS, KP_DEL.VSS, KP_DELETE2.VSS, KP_SLASH.VSS, L.VSS, LBRACKET.VSS, LEFT.VSS, LOCK.VSS, M.VSS, M2.VSS, M3.VSS, M4.VSS, M5.VSS, M6.VSS, MENU.VSS, N.VSS, NEXTSONG.VSS, NUMLOCK.VSS, O.VSS, P.VSS, PAUSE.VSS, PAUSEPLAY.VSS, PERIOD.VSS, PGDN.VSS, PGUP.VSS, PLUS2.VSS, PRTSC.VSS, Q.VSS, QUOTE.VSS, R.VSS, RANDSONG.VSS, RBRACKET.VSS, RIGHT.VSS, S.VSS, SCROLLLOCK.VSS, SEMICOLON.VSS, SHIFT.VSS, SHIFT2.VSS, SLASH.VSS, SPACE.B-, T.VSS, TAB.VSS, U.VSS, UNDERSCORE.VSS, UP.VSS, V.VSS, VOLUMEUP.VSS, VOLUMNEDOWN.VSS, W.VSS, WIN.VSS, WIN2.VSS, X.VSS, Y.VSS, Z.VSS
- net LED1: now also IC3.54
- net LED2: now also IC3.55
- net LED3: now also IC3.56
- net LED4: now also IC3.57
- net LED5: now also IC3.58
- net LED6: now also IC3.59
- net N$164: now also BACKSPACE.DOUT; no longer BACKSPACE.G-
- net N$193: now also PLUS2.DIN; no longer EQUAL2.DIN
- net N$194: now also PLUS2.DOUT; no longer EQUAL2.DOUT
- net N$207: now also ENTER.DIN; no longer ENTER.R-
- net N$208: now also ENTER.DOUT; no longer ENTER.G-
- net N$214: now also SHIFT.DIN; no longer SHIFT.R-
- net N$215: now also SHIFT.DOUT; no longer SHIFT.G-
- net N$225: now also SHIFT2.DIN; no longer SHIFT2.R-
- net N$230: now also SHIFT2.DOUT; no longer SHIFT2.G-
- net N$247: now also KP_0.DIN; no longer KP_0.R-
- net N$248: now also KP_0.DOUT; no longer KP_0.G-
- net N$65: now also PLUS2.ALPS2, PLUS2.MX2; no longer EQUAL2.ALPS2, EQUAL2.MX2
- net ROW1: now also IC3.15
- net ROW2: now also IC3.14
- net ROW3: now also IC3.13
- net ROW4: now also IC3.12
- net ROW5: now also IC3.11
- net ROW6: now also DCTRL.C, IC3.10
Routing:
- net +5V: track 93.4 -> 886.8 mm, vias 7 -> 18
- net GND: track 151.9 -> 750.0 mm, vias 4 -> 6
- net LED6: track 0.00 -> 573.1 mm
- net LED5: track 0.00 -> 552.1 mm
- net LED4: track 0.00 -> 530.7 mm
- net ROW2: track 0.00 -> 518.0 mm
- net LED3: track 0.00 -> 508.9 mm
- net LED2: track 0.00 -> 487.5 mm
- net ROW1: track 0.00 -> 480.5 mm
- net LED1: track 0.00 -> 466.2 mm
- net COL2: track 0.00 -> 436.7 mm, vias 0 -> 1
- net COL3: track 0.00 -> 415.5 mm, vias 0 -> 1
- net COL4: track 0.00 -> 393.8 mm, vias 0 -> 1
- net COL5: track 0.00 -> 374.3 mm, vias 0 -> 1
- net COL6: track 0.00 -> 354.9 mm, vias 0 -> 1
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Other:
- board size 487.7 x 175.3 mm -> 485.6 x 151 mm

Commit message: Updated keyboard schematic. Slowely making progress
Parts:
- moved DBACKSLASH 1.05 mm to (276.8, 72.4)
- moved DRBRACKET 1.02 mm to (252.8, 72.4)
Connections:
- net +5V: now also F8.VDD, SPACE.VDD, VOLUMNEDOWN.VDD; no longer SPACE.LED+
- net GND: now also SPACE.VSS; no longer SPACE.B-
- net N$235: now also SPACE.DIN; no longer SPACE.R-
- net N$238: now also SPACE.DOUT; no longer SPACE.G-
Routing:
- net GND: track 750.0 -> 3713.8 mm, vias 6 -> 16
- net +5V: track 886.8 -> 3766.9 mm, vias 18 -> 61
- net COL2: track 436.7 -> 557.5 mm, vias 1 -> 6
- net N$214: track 0.00 -> 27.4 mm
- net N$195: track 0.00 -> 22.7 mm
- net N$172: track 0.00 -> 20.3 mm
- net N$232: track 0.00 -> 17.9 mm
- net N$149: track 0.00 -> 15.6 mm
- net N$135: track 0.00 -> 15.5 mm
- net N$136: track 0.00 -> 15.5 mm
- net N$134: track 0.00 -> 15.5 mm
- net N$133: track 0.00 -> 15.5 mm
- net N$124: track 0.00 -> 15.5 mm
- net N$121: track 0.00 -> 15.5 mm
- net N$132: track 0.00 -> 15.5 mm
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
Commit message: Updated before rework of keys
Parts:
- moved DSHIFT2 2.34 mm to (274.6, 37.4)
- moved DCTRL 1.05 mm to (16.8, 18.6)
- moved DM1 1.05 mm to (-4.67, 18.6)
- moved D0 1.02 mm to (205.1, 94.8)
- moved D1 1.02 mm to (33.7, 94.8)
- moved D2 1.02 mm to (52.7, 94.8)
- moved D3 1.02 mm to (71.8, 94.8)
- moved D4 1.02 mm to (90.8, 94.8)
- moved D5 1.02 mm to (109.9, 94.8)
- moved D6 1.02 mm to (128.9, 94.8)
- moved D7 1.02 mm to (148.0, 94.8)
- moved D8 1.02 mm to (167.0, 94.8)
- moved D9 1.02 mm to (186.1, 94.8)
- moved DBACKSPACE 1.02 mm to (271.8, 94.8)
- moved DDASH 1.02 mm to (224.2, 94.8)
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Connections:
- new net N$117: SHIFT2.DOUT, UP.DIN
- net +5V: now also KP_2.VDD, SHIFT2.VDD
- net N$230: now also UP.DOUT; no longer SHIFT2.DOUT
Routing:
- net +5V: track 3766.9 -> 4375.2 mm, vias 61 -> 126
- net ROW6: track 149.7 -> 602.9 mm
- net ROW4: track 108.3 -> 556.4 mm, vias 0 -> 2
- net ROW5: track 128.8 -> 572.7 mm
- net ROW3: track 87.5 -> 525.8 mm
- net COL4: track 393.8 -> 548.6 mm, vias 1 -> 7
- net COL5: track 374.3 -> 516.6 mm, vias 1 -> 6
- net COL13: track 217.0 -> 355.0 mm, vias 1 -> 6
- net COL8: track 316.4 -> 454.3 mm, vias 1 -> 6
- net COL12: track 236.3 -> 370.8 mm, vias 1 -> 6
- net COL3: track 415.5 -> 546.0 mm, vias 1 -> 6
- net COL6: track 354.9 -> 469.7 mm, vias 1 -> 5
- net COL11: track 255.7 -> 370.1 mm, vias 1 -> 5
- net COL9: track 294.7 -> 408.3 mm, vias 1 -> 5
- net COL7: track 335.7 -> 449.3 mm, vias 1 -> 5
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Other:
- board size 485.6 x 151 mm -> 479 x 151.7 mm

Commit message: blank reverse
Parts:
- moved J1 458.0 mm to (-18.3, 141.5), flipped to the top
- moved R6 451.2 mm to (-14.9, 147.8), flipped to the top
- moved S1 447.3 mm to (-13.0, 130.3), flipped to the top
- moved R5 442.7 mm to (-10.6, 143.2), flipped to the top
- moved R3 441.3 mm to (-9.96, 140.2), flipped to the top
- moved R4 441.3 mm to (-9.96, 138.2), flipped to the top
- moved C5 421.4 mm to (0.00, 135.6), flipped to the top
- moved C7 421.4 mm to (0.00, 143.8), flipped to the top
- moved C8 421.4 mm to (0.00, 137.7), flipped to the top
- moved R1 417.3 mm to (2.06, 124.3), flipped to the top
- moved C4 413.2 mm to (4.09, 124.3), flipped to the top
- moved C3 412.3 mm to (4.57, 145.1), flipped to the top
- moved C2 406.2 mm to (7.62, 124.2), flipped to the top
- moved Y2 400.1 mm to (10.7, 124.2), flipped to the top
- moved IC3 396.0 mm to (12.7, 136.1), flipped to the top
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Connections:
- net +5V: now also ENTER2.DOUT, KP_0.DOUT, PLUS2.DOUT, SHIFT.DOUT, SHIFT2.DOUT, SPACE.DOUT; no longer ENTER2.VDD, KP_0.VDD, PLUS2.VDD, SHIFT.VDD, SHIFT2.VDD, SPACE.VDD
- net COL10: now also 7.ALPS2, 7.MX2, F7.ALPS2, F7.MX2, J.ALPS2, J.MX2, M.ALPS2, M.MX2, U.ALPS2, U.MX2; no longer 7.ALPS1, 7.MX1, F7.ALPS1, F7.MX1, J.ALPS1, J.MX1, M.ALPS1, M.MX1, U.ALPS1, U.MX1
- net COL11: now also 8.ALPS2, 8.MX2, COMMA.ALPS2, COMMA.MX2, F8.ALPS2, F8.MX2, I.ALPS2, I.MX2, K.ALPS2, K.MX2; no longer 8.ALPS1, 8.MX1, COMMA.ALPS1, COMMA.MX1, F8.ALPS1, F8.MX1, I.ALPS1, I.MX1, K.ALPS1, K.MX1
- net COL12: now also 9.ALPS2, 9.MX2, ALT2.ALPS2, ALT2.MX2, F9.ALPS2, F9.MX2, L.ALPS2, L.MX2, O.ALPS2, O.MX2, PERIOD.ALPS2, PERIOD.MX2; no longer 9.ALPS1, 9.MX1, ALT2.ALPS1, ALT2.MX1, F9.ALPS1, F9.MX1, L.ALPS1, L.MX1, O.ALPS1, O.MX1, PERIOD.ALPS1, PERIOD.MX1
- net COL13: now also 0.ALPS2, 0.MX2, F10.ALPS2, F10.MX2, P.ALPS2, P.MX2, SEMICOLON.ALPS2, SEMICOLON.MX2, SLASH.ALPS2, SLASH.MX2, WIN2.ALPS2, WIN2.MX2; no longer 0.ALPS1, 0.MX1, F10.ALPS1, F10.MX1, P.ALPS1, P.MX1, SEMICOLON.ALPS1, SEMICOLON.MX1, SLASH.ALPS1, SLASH.MX1, WIN2.ALPS1, WIN2.MX1
- net COL14: now also DASH.ALPS2, DASH.MX2, F11.ALPS2, F11.MX2, LBRACKET.ALPS2, LBRACKET.MX2, MENU.ALPS2, MENU.MX2, QUOTE.ALPS2, QUOTE.MX2; no longer DASH.ALPS1, DASH.MX1, F11.ALPS1, F11.MX1, LBRACKET.ALPS1, LBRACKET.MX1, MENU.ALPS1, MENU.MX1, QUOTE.ALPS1, QUOTE.MX1
- net COL15: now also EQUAL.ALPS2, EQUAL.MX2, F12.ALPS2, F12.MX2, RBRACKET.ALPS2, RBRACKET.MX2; no longer EQUAL.ALPS1, EQUAL.MX1, F12.ALPS1, F12.MX1, RBRACKET.ALPS1, RBRACKET.MX1
- net COL16: now also VOLUMEUP.ALPS2, VOLUMEUP.MX2; no longer VOLUMEUP.ALPS1, VOLUMEUP.MX1
- net COL17: now also BACKSLASH.ALPS2, BACKSLASH.MX2, BACKSPACE.ALPS2, BACKSPACE.MX2, CTRL2.ALPS2, CTRL2.MX2, ENTER.ALPS2, ENTER.MX2, SHIFT2.ALPS2, SHIFT2.MX2, VOLUMNEDOWN.ALPS2, VOLUMNEDOWN.MX2; no longer BACKSLASH.ALPS1, BACKSLASH.MX1, BACKSPACE.ALPS1, BACKSPACE.MX1, CTRL2.ALPS1, CTRL2.MX1, ENTER.ALPS1, ENTER.MX1, SHIFT2.ALPS1, SHIFT2.MX1, VOLUMNEDOWN.ALPS1, VOLUMNEDOWN.MX1
- net COL18: now also DELETE.ALPS2, DELETE.MX2, INSERT.ALPS2, INSERT.MX2, LEFT.ALPS2, LEFT.MX2, PRTSC.ALPS2, PRTSC.MX2; no longer DELETE.ALPS1, DELETE.MX1, INSERT.ALPS1, INSERT.MX1, LEFT.ALPS1, LEFT.MX1, PRTSC.ALPS1, PRTSC.MX1
- net COL19: now also DOWN.ALPS2, DOWN.MX2, END.ALPS2, END.MX2, HOME.ALPS2, HOME.MX2, SCROLLLOCK.ALPS2, SCROLLLOCK.MX2, UP.ALPS2, UP.MX2; no longer DOWN.ALPS1, DOWN.MX1, END.ALPS1, END.MX1, HOME.ALPS1, HOME.MX1, SCROLLLOCK.ALPS1, SCROLLLOCK.MX1, UP.ALPS1, UP.MX1
- net COL2: now also CTRL1.ALPS2, CTRL1.MX2, M2.ALPS2, M2.MX2, M3.ALPS2, M3.MX2, M4.ALPS2, M4.MX2, M5.ALPS2, M5.MX2, M6.ALPS2, M6.MX2; no longer CTRL1.ALPS1, CTRL1.MX1, M2.ALPS1, M2.MX1, M3.ALPS1, M3.MX1, M4.ALPS1, M4.MX1, M5.ALPS1, M5.MX1, M6.ALPS1, M6.MX1
- net COL20: now also PAUSE.ALPS2, PAUSE.MX2, PGDN.ALPS2, PGDN.MX2, PGUP.ALPS2, PGUP.MX2, RIGHT.ALPS2, RIGHT.MX2; no longer PAUSE.ALPS1, PAUSE.MX1, PGDN.ALPS1, PGDN.MX1, PGUP.ALPS1, PGUP.MX1, RIGHT.ALPS1, RIGHT.MX1
- net COL21: now also BACKSONG.ALPS2, BACKSONG.MX2, KP_0.ALPS2, KP_0.MX2, KP_1.ALPS2, KP_1.MX2, KP_4.ALPS2, KP_4.MX2, KP_7.ALPS2, KP_7.MX2, NUMLOCK.ALPS2, NUMLOCK.MX2; no longer BACKSONG.ALPS1, BACKSONG.MX1, KP_0.ALPS1, KP_0.MX1, KP_1.ALPS1, KP_1.MX1, KP_4.ALPS1, KP_4.MX1, KP_7.ALPS1, KP_7.MX1, NUMLOCK.ALPS1, NUMLOCK.MX1
- net COL22: now also KP_2.ALPS2, KP_2.MX2, KP_52.ALPS2, KP_52.MX2, KP_8.ALPS2, KP_8.MX2, KP_SLASH.ALPS2, KP_SLASH.MX2, PAUSEPLAY.ALPS2, PAUSEPLAY.MX2; no longer KP_2.ALPS1, KP_2.MX1, KP_52.ALPS1, KP_52.MX1, KP_8.ALPS1, KP_8.MX1, KP_SLASH.ALPS1, KP_SLASH.MX1, PAUSEPLAY.ALPS1, PAUSEPLAY.MX1
- net COL23: now also KP_3.ALPS2, KP_3.MX2, KP_6.ALPS2, KP_6.MX2, KP_9.ALPS2, KP_9.MX2, KP_ASTERISK.ALPS2, KP_ASTERISK.MX2, KP_DEL.ALPS2, KP_DEL.MX2, NEXTSONG.ALPS2, NEXTSONG.MX2; no longer KP_3.ALPS1, KP_3.MX1, KP_6.ALPS1, KP_6.MX1, KP_9.ALPS1, KP_9.MX1, KP_ASTERISK.ALPS1, KP_ASTERISK.MX1, KP_DEL.ALPS1, KP_DEL.MX1, NEXTSONG.ALPS1, NEXTSONG.MX1
- net COL24: now also ENTER2.ALPS2, ENTER2.MX2, KP_DASH.ALPS2, KP_DASH.MX2, PLUS2.ALPS2, PLUS2.MX2, RANDSONG.ALPS2, RANDSONG.MX2; no longer ENTER2.ALPS1, ENTER2.MX1, KP_DASH.ALPS1, KP_DASH.MX1, PLUS2.ALPS1, PLUS2.MX1, RANDSONG.ALPS1, RANDSONG.MX1
- net COL25: now also BACKSPACE_1.ALPS2, BACKSPACE_1.MX2, KP_5.ALPS2, KP_5.MX2, KP_62.ALPS2, KP_62.MX2, KP_DELETE2.ALPS2, KP_DELETE2.MX2, LOCK.ALPS2, LOCK.MX2, UNDERSCORE.ALPS2, UNDERSCORE.MX2; no longer BACKSPACE_1.ALPS1, BACKSPACE_1.MX1, KP_5.ALPS1, KP_5.MX1, KP_62.ALPS1, KP_62.MX1, KP_DELETE2.ALPS1, KP_DELETE2.MX1, LOCK.ALPS1, LOCK.MX1, UNDERSCORE.ALPS1, UNDERSCORE.MX1
- net COL3: now also CAPSLOCK.ALPS2, CAPSLOCK.MX2, CTRL.ALPS2, CTRL.MX2, ESC.ALPS2, ESC.MX2, GRAVE.ALPS2, GRAVE.MX2, SHIFT.ALPS2, SHIFT.MX2, TAB.ALPS2, TAB.MX2; no longer CAPSLOCK.ALPS1, CAPSLOCK.MX1, CTRL.ALPS1, CTRL.MX1, ESC.ALPS1, ESC.MX1, GRAVE.ALPS1, GRAVE.MX1, SHIFT.ALPS1, SHIFT.MX1, TAB.ALPS1, TAB.MX1
- net COL4: now also 1.ALPS2, 1.MX2, A.ALPS2, A.MX2, F1.ALPS2, F1.MX2, Q.ALPS2, Q.MX2, WIN.ALPS2, WIN.MX2, Z.ALPS2, Z.MX2; no longer 1.ALPS1, 1.MX1, A.ALPS1, A.MX1, F1.ALPS1, F1.MX1, Q.ALPS1, Q.MX1, WIN.ALPS1, WIN.MX1, Z.ALPS1, Z.MX1
- net COL5: now also 2.ALPS2, 2.MX2, ALT.ALPS2, ALT.MX2, F2.ALPS2, F2.MX2, S.ALPS2, S.MX2, W.ALPS2, W.MX2, X.ALPS2, X.MX2; no longer 2.ALPS1, 2.MX1, ALT.ALPS1, ALT.MX1, F2.ALPS1, F2.MX1, S.ALPS1, S.MX1, W.ALPS1, W.MX1, X.ALPS1, X.MX1
- net COL6: now also 3.ALPS2, 3.MX2, C.ALPS2, C.MX2, D.ALPS2, D.MX2, E.ALPS2, E.MX2, F3.ALPS2, F3.MX2; no longer 3.ALPS1, 3.MX1, C.ALPS1, C.MX1, D.ALPS1, D.MX1, E.ALPS1, E.MX1, F3.ALPS1, F3.MX1
- net COL7: now also 4.ALPS2, 4.MX2, F.ALPS2, F.MX2, F4.ALPS2, F4.MX2, R.ALPS2, R.MX2, V.ALPS2, V.MX2; no longer 4.ALPS1, 4.MX1, F.ALPS1, F.MX1, F4.ALPS1, F4.MX1, R.ALPS1, R.MX1, V.ALPS1, V.MX1
- net COL8: now also 5.ALPS2, 5.MX2, B.ALPS2, B.MX2, F5.ALPS2, F5.MX2, G.ALPS2, G.MX2, SPACE.ALPS2, SPACE.MX2, T.ALPS2, T.MX2; no longer 5.ALPS1, 5.MX1, B.ALPS1, B.MX1, F5.ALPS1, F5.MX1, G.ALPS1, G.MX1, SPACE.ALPS1, SPACE.MX1, T.ALPS1, T.MX1
- net COL9: now also 6.ALPS2, 6.MX2, F6.ALPS2, F6.MX2, H.ALPS2, H.MX2, N.ALPS2, N.MX2, Y.ALPS2, Y.MX2; no longer 6.ALPS1, 6.MX1, F6.ALPS1, F6.MX1, H.ALPS1, H.MX1, N.ALPS1, N.MX1, Y.ALPS1, Y.MX1
- net GND: now also BACKSPACE.DIN, ENTER.DIN, ENTER2.DIN, KP_0.DIN, PLUS2.DIN, SHIFT.DIN, SHIFT2.DIN, SPACE.DIN; no longer BACKSPACE.VSS, ENTER.VSS, ENTER2.VSS, KP_0.VSS, PLUS2.VSS, SHIFT.VSS, SHIFT2.VSS, SPACE.VSS
- net LED1: now also IC3.15; no longer IC3.54
- net LED2: now also IC3.14; no longer IC3.55
- net LED3: now also IC3.13; no longer IC3.56
- net LED4: now also IC3.12; no longer IC3.57
- net LED5: now also IC3.11; no longer IC3.58
- net LED6: now also IC3.10; no longer IC3.59
- net N$1: now also ESC.ALPS1, ESC.MX1; no longer ESC.ALPS2, ESC.MX2
- net N$10: now also F9.ALPS1, F9.MX1; no longer F9.ALPS2, F9.MX2
- net N$100: now also ENTER2.ALPS1, ENTER2.MX1; no longer ENTER2.ALPS2, ENTER2.MX2
- net N$101: now also KP_DELETE2.ALPS1, KP_DELETE2.MX1; no longer KP_DELETE2.ALPS2, KP_DELETE2.MX2
- net N$102: now also CTRL.ALPS1, CTRL.MX1; no longer CTRL.ALPS2, CTRL.MX2
- net N$103: now also WIN.ALPS1, WIN.MX1; no longer WIN.ALPS2, WIN.MX2
- net N$104: now also ALT.ALPS1, ALT.MX1; no longer ALT.ALPS2, ALT.MX2
- net N$105: now also SPACE.ALPS1, SPACE.MX1; no longer SPACE.ALPS2, SPACE.MX2
- net N$106: now also ALT2.ALPS1, ALT2.MX1; no longer ALT2.ALPS2, ALT2.MX2
- net N$108: now also MENU.ALPS1, MENU.MX1; no longer MENU.ALPS2, MENU.MX2
- net N$109: now also CTRL2.ALPS1, CTRL2.MX1; no longer CTRL2.ALPS2, CTRL2.MX2
- net N$11: now also F10.ALPS1, F10.MX1; no longer F10.ALPS2, F10.MX2
- net N$110: now also LEFT.ALPS1, LEFT.MX1; no longer LEFT.ALPS2, LEFT.MX2
- net N$111: now also DOWN.ALPS1, DOWN.MX1; no longer DOWN.ALPS2, DOWN.MX2
- net N$112: now also RIGHT.ALPS1, RIGHT.MX1; no longer RIGHT.ALPS2, RIGHT.MX2
- net N$113: now also KP_0.ALPS1, KP_0.MX1; no longer KP_0.ALPS2, KP_0.MX2
- net N$114: now also KP_DEL.ALPS1, KP_DEL.MX1; no longer KP_DEL.ALPS2, KP_DEL.MX2
- net N$115: now also BACKSPACE_1.ALPS1, BACKSPACE_1.MX1; no longer BACKSPACE_1.ALPS2, BACKSPACE_1.MX2
- net N$116: now also BACKSPACE.VSS; no longer BACKSPACE.DIN
- net N$117: now also SHIFT2.VDD; no longer SHIFT2.DOUT
- net N$12: now also F11.ALPS1, F11.MX1; no longer F11.ALPS2, F11.MX2
- net N$120: now also M6.ALPS1, M6.MX1; no longer M6.ALPS2, M6.MX2
- net N$125: now also WIN2.ALPS1, WIN2.MX1; no longer WIN2.ALPS2, WIN2.MX2
- net N$126: now also M2.ALPS1, M2.MX1; no longer M2.ALPS2, M2.MX2
- net N$127: now also M5.ALPS1, M5.MX1; no longer M5.ALPS2, M5.MX2
- net N$128: now also M4.ALPS1, M4.MX1; no longer M4.ALPS2, M4.MX2
- net N$129: now also M3.ALPS1, M3.MX1; no longer M3.ALPS2, M3.MX2
- net N$13: now also F12.ALPS1, F12.MX1; no longer F12.ALPS2, F12.MX2
- net N$130: now also CTRL1.ALPS1, CTRL1.MX1; no longer CTRL1.ALPS2, CTRL1.MX2
- net N$131: now also RANDSONG.ALPS1, RANDSONG.MX1; no longer RANDSONG.ALPS2, RANDSONG.MX2
- net N$14: now also VOLUMEUP.ALPS1, VOLUMEUP.MX1; no longer VOLUMEUP.ALPS2, VOLUMEUP.MX2
- net N$15: now also VOLUMNEDOWN.ALPS1, VOLUMNEDOWN.MX1; no longer VOLUMNEDOWN.ALPS2, VOLUMNEDOWN.MX2
- net N$16: now also PRTSC.ALPS1, PRTSC.MX1; no longer PRTSC.ALPS2, PRTSC.MX2
- net N$164: now also BACKSPACE.VDD; no longer BACKSPACE.DOUT
- net N$17: now also SCROLLLOCK.ALPS1, SCROLLLOCK.MX1; no longer SCROLLLOCK.ALPS2, SCROLLLOCK.MX2
- net N$18: now also PAUSE.ALPS1, PAUSE.MX1; no longer PAUSE.ALPS2, PAUSE.MX2
- net N$19: now also BACKSONG.ALPS1, BACKSONG.MX1; no longer BACKSONG.ALPS2, BACKSONG.MX2
- net N$193: now also PLUS2.VSS; no longer PLUS2.DIN
- net N$194: now also PLUS2.VDD; no longer PLUS2.DOUT
- net N$2: now also F1.ALPS1, F1.MX1; no longer F1.ALPS2, F1.MX2
- net N$20: now also PAUSEPLAY.ALPS1, PAUSEPLAY.MX1; no longer PAUSEPLAY.ALPS2, PAUSEPLAY.MX2
- net N$207: now also ENTER.VSS; no longer ENTER.DIN
- net N$208: now also ENTER.VDD; no longer ENTER.DOUT
- net N$209: now also ENTER2.VSS; no longer ENTER2.DIN
- net N$21: now also NEXTSONG.ALPS1, NEXTSONG.MX1; no longer NEXTSONG.ALPS2, NEXTSONG.MX2
- net N$214: now also SHIFT.VSS; no longer SHIFT.DIN
- net N$215: now also SHIFT.VDD; no longer SHIFT.DOUT
- net N$22: now also LOCK.ALPS1, LOCK.MX1; no longer LOCK.ALPS2, LOCK.MX2
- net N$225: now also SHIFT2.VSS; no longer SHIFT2.DIN
- net N$229: now also ENTER2.VDD; no longer ENTER2.DOUT
- net N$23: now also GRAVE.ALPS1, GRAVE.MX1; no longer GRAVE.ALPS2, GRAVE.MX2
- net N$235: now also SPACE.VSS; no longer SPACE.DIN
- net N$238: now also SPACE.VDD; no longer SPACE.DOUT
- net N$24: now also 1.ALPS1, 1.MX1; no longer 1.ALPS2, 1.MX2
- net N$247: now also KP_0.VSS; no longer KP_0.DIN
- net N$248: now also KP_0.VDD; no longer KP_0.DOUT
- net N$25: now also 2.ALPS1, 2.MX1; no longer 2.ALPS2, 2.MX2
- net N$26: now also 3.ALPS1, 3.MX1; no longer 3.ALPS2, 3.MX2
- net N$27: now also 4.ALPS1, 4.MX1; no longer 4.ALPS2, 4.MX2
- net N$28: now also 5.ALPS1, 5.MX1; no longer 5.ALPS2, 5.MX2
- net N$29: now also 6.ALPS1, 6.MX1; no longer 6.ALPS2, 6.MX2
- net N$3: now also F2.ALPS1, F2.MX1; no longer F2.ALPS2, F2.MX2
- net N$30: now also 7.ALPS1, 7.MX1; no longer 7.ALPS2, 7.MX2
- net N$31: now also 8.ALPS1, 8.MX1; no longer 8.ALPS2, 8.MX2
- net N$32: now also 9.ALPS1, 9.MX1; no longer 9.ALPS2, 9.MX2
- net N$33: now also 0.ALPS1, 0.MX1; no longer 0.ALPS2, 0.MX2
- net N$34: now also DASH.ALPS1, DASH.MX1; no longer DASH.ALPS2, DASH.MX2
- net N$35: now also EQUAL.ALPS1, EQUAL.MX1; no longer EQUAL.ALPS2, EQUAL.MX2
- net N$36: now also BACKSPACE.ALPS1, BACKSPACE.MX1; no longer BACKSPACE.ALPS2, BACKSPACE.MX2
- net N$37: now also INSERT.ALPS1, INSERT.MX1; no longer INSERT.ALPS2, INSERT.MX2
- net N$38: now also HOME.ALPS1, HOME.MX1; no longer HOME.ALPS2, HOME.MX2
- net N$39: now also PGUP.ALPS1, PGUP.MX1; no longer PGUP.ALPS2, PGUP.MX2
- net N$4: now also F3.ALPS1, F3.MX1; no longer F3.ALPS2, F3.MX2
- net N$40: now also NUMLOCK.ALPS1, NUMLOCK.MX1; no longer NUMLOCK.ALPS2, NUMLOCK.MX2
- net N$41: now also KP_SLASH.ALPS1, KP_SLASH.MX1; no longer KP_SLASH.ALPS2, KP_SLASH.MX2
- net N$42: now also KP_ASTERISK.ALPS1, KP_ASTERISK.MX1; no longer KP_ASTERISK.ALPS2, KP_ASTERISK.MX2
- net N$43: now also KP_DASH.ALPS1, KP_DASH.MX1; no longer KP_DASH.ALPS2, KP_DASH.MX2
- net N$44: now also UNDERSCORE.ALPS1, UNDERSCORE.MX1; no longer UNDERSCORE.ALPS2, UNDERSCORE.MX2
- net N$45: now also TAB.ALPS1, TAB.MX1; no longer TAB.ALPS2, TAB.MX2
- net N$46: now also Q.ALPS1, Q.MX1; no longer Q.ALPS2, Q.MX2
- net N$47: now also W.ALPS1, W.MX1; no longer W.ALPS2, W.MX2
- net N$48: now also E.ALPS1, E.MX1; no longer E.ALPS2, E.MX2
- net N$49: now also R.ALPS1, R.MX1; no longer R.ALPS2, R.MX2
- net N$5: now also F4.ALPS1, F4.MX1; no longer F4.ALPS2, F4.MX2
- net N$50: now also T.ALPS1, T.MX1; no longer T.ALPS2, T.MX2
- net N$51: now also Y.ALPS1, Y.MX1; no longer Y.ALPS2, Y.MX2
- net N$52: now also U.ALPS1, U.MX1; no longer U.ALPS2, U.MX2
- net N$53: now also I.ALPS1, I.MX1; no longer I.ALPS2, I.MX2
- net N$54: now also O.ALPS1, O.MX1; no longer O.ALPS2, O.MX2
- net N$55: now also P.ALPS1, P.MX1; no longer P.ALPS2, P.MX2
- net N$56: now also LBRACKET.ALPS1, LBRACKET.MX1; no longer LBRACKET.ALPS2, LBRACKET.MX2
- net N$57: now also RBRACKET.ALPS1, RBRACKET.MX1; no longer RBRACKET.ALPS2, RBRACKET.MX2
- net N$58: now also BACKSLASH.ALPS1, BACKSLASH.MX1; no longer BACKSLASH.ALPS2, BACKSLASH.MX2
- net N$59: now also DELETE.ALPS1, DELETE.MX1; no longer DELETE.ALPS2, DELETE.MX2
- net N$6: now also F5.ALPS1, F5.MX1; no longer F5.ALPS2, F5.MX2
- net N$60: now also END.ALPS1, END.MX1; no longer END.ALPS2, END.MX2
- net N$61: now also PGDN.ALPS1, PGDN.MX1; no longer PGDN.ALPS2, PGDN.MX2
- net N$62: now also KP_7.ALPS1, KP_7.MX1; no longer KP_7.ALPS2, KP_7.MX2
- net N$63: now also KP_8.ALPS1, KP_8.MX1; no longer KP_8.ALPS2, KP_8.MX2
- net N$64: now also KP_9.ALPS1, KP_9.MX1; no longer KP_9.ALPS2, KP_9.MX2
- net N$65: now also PLUS2.ALPS1, PLUS2.MX1; no longer PLUS2.ALPS2, PLUS2.MX2
- net N$66: now also KP_5.ALPS1, KP_5.MX1; no longer KP_5.ALPS2, KP_5.MX2
- net N$67: now also CAPSLOCK.ALPS1, CAPSLOCK.MX1; no longer CAPSLOCK.ALPS2, CAPSLOCK.MX2
- net N$68: now also A.ALPS1, A.MX1; no longer A.ALPS2, A.MX2
- net N$69: now also S.ALPS1, S.MX1; no longer S.ALPS2, S.MX2
- net N$7: now also F6.ALPS1, F6.MX1; no longer F6.ALPS2, F6.MX2
- net N$70: now also D.ALPS1, D.MX1; no longer D.ALPS2, D.MX2
- net N$71: now also F.ALPS1, F.MX1; no longer F.ALPS2, F.MX2
- net N$72: now also G.ALPS1, G.MX1; no longer G.ALPS2, G.MX2
- net N$73: now also H.ALPS1, H.MX1; no longer H.ALPS2, H.MX2
- net N$74: now also J.ALPS1, J.MX1; no longer J.ALPS2, J.MX2
- net N$75: now also K.ALPS1, K.MX1; no longer K.ALPS2, K.MX2
- net N$76: now also L.ALPS1, L.MX1; no longer L.ALPS2, L.MX2
- net N$77: now also SEMICOLON.ALPS1, SEMICOLON.MX1; no longer SEMICOLON.ALPS2, SEMICOLON.MX2
- net N$78: now also QUOTE.ALPS1, QUOTE.MX1; no longer QUOTE.ALPS2, QUOTE.MX2
- net N$79: now also ENTER.ALPS1, ENTER.MX1; no longer ENTER.ALPS2, ENTER.MX2
- net N$8: now also F7.ALPS1, F7.MX1; no longer F7.ALPS2, F7.MX2
- net N$80: now also KP_4.ALPS1, KP_4.MX1; no longer KP_4.ALPS2, KP_4.MX2
- net N$81: now also KP_52.ALPS1, KP_52.MX1; no longer KP_52.ALPS2, KP_52.MX2
- net N$82: now also KP_6.ALPS1, KP_6.MX1; no longer KP_6.ALPS2, KP_6.MX2
- net N$83: now also KP_62.ALPS1, KP_62.MX1; no longer KP_62.ALPS2, KP_62.MX2
- net N$84: now also SHIFT.ALPS1, SHIFT.MX1; no longer SHIFT.ALPS2, SHIFT.MX2
- net N$85: now also Z.ALPS1, Z.MX1; no longer Z.ALPS2, Z.MX2
- net N$86: now also X.ALPS1, X.MX1; no longer X.ALPS2, X.MX2
- net N$87: now also C.ALPS1, C.MX1; no longer C.ALPS2, C.MX2
- net N$88: now also V.ALPS1, V.MX1; no longer V.ALPS2, V.MX2
- net N$89: now also B.ALPS1, B.MX1; no longer B.ALPS2, B.MX2
- net N$9: now also F8.ALPS1, F8.MX1; no longer F8.ALPS2, F8.MX2
- net N$90: now also N.ALPS1, N.MX1; no longer N.ALPS2, N.MX2
- net N$91: now also M.ALPS1, M.MX1; no longer M.ALPS2, M.MX2
- net N$92: now also COMMA.ALPS1, COMMA.MX1; no longer COMMA.ALPS2, COMMA.MX2
- net N$93: now also PERIOD.ALPS1, PERIOD.MX1; no longer PERIOD.ALPS2, PERIOD.MX2
- net N$94: now also SLASH.ALPS1, SLASH.MX1; no longer SLASH.ALPS2, SLASH.MX2
- net N$95: now also SHIFT2.ALPS1, SHIFT2.MX1; no longer SHIFT2.ALPS2, SHIFT2.MX2
- net N$96: now also UP.ALPS1, UP.MX1; no longer UP.ALPS2, UP.MX2
- net N$97: now also KP_1.ALPS1, KP_1.MX1; no longer KP_1.ALPS2, KP_1.MX2
- net N$98: now also KP_2.ALPS1, KP_2.MX1; no longer KP_2.ALPS2, KP_2.MX2
- net N$99: now also KP_3.ALPS1, KP_3.MX1; no longer KP_3.ALPS2, KP_3.MX2
- net ROW1: now also IC3.54; no longer IC3.15
- net ROW2: now also IC3.55; no longer IC3.14
- net ROW3: now also IC3.56; no longer IC3.13
- net ROW4: now also IC3.57; no longer IC3.12
- net ROW5: now also IC3.58; no longer IC3.11
- net ROW6: now also IC3.59; no longer IC3.10
Routing:
- net +5V: track 4375.2 -> 93.5 mm, vias 126 -> 7
- net GND: track 3780.9 -> 151.7 mm, vias 16 -> 4
- net ROW6: track 602.9 -> 0.00 mm
- net ROW5: track 572.7 -> 0.00 mm
- net LED6: track 574.4 -> 5.69 mm
- net COL2: track 557.5 -> 0.00 mm, vias 6 -> 0
- net ROW4: track 556.4 -> 0.00 mm, vias 2 -> 0
- net COL4: track 548.6 -> 0.00 mm, vias 7 -> 0
- net LED5: track 553.4 -> 4.86 mm
- net COL3: track 546.0 -> 0.00 mm, vias 6 -> 0
- net LED4: track 531.9 -> 4.18 mm
- net ROW3: track 525.8 -> 0.00 mm
- net COL5: track 516.6 -> 0.00 mm, vias 6 -> 0
- net LED3: track 510.1 -> 3.85 mm
- net ROW2: track 506.2 -> 0.00 mm
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