File: EAGLE_PCB/keyboard.sch (EAGLE design)
At the start: 262 parts, among them J1 1-2295018-2, M2 KEYSWITCH-RGBSMDLED-ALPSMX-1U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, M3 KEYSWITCH-RGBSMDLED-ALPSMX-1U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, M4 KEYSWITCH-RGBSMDLED-ALPSMX-1U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, M5 KEYSWITCH-RGBSMDLED-ALPSMX-1U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, M6 KEYSWITCH-RGBSMDLED-ALPSMX-1U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, Y2 CRYSTAL-GROUNDEDSMD-3.2X2.5

Commit message: Updated alot might switch to kicad
Connections:
- net +5V: now also BACKSLASH.VCC, BACKSPACE.VCC, KP_2.VCC, KP_8.VCC, KP_SLASH.VCC, SHIFT2.VCC
Other:
- moved on the sheet: ENTER2, PLUS2
