File: EAGLE_PCB_V2/board.brd (EAGLE design)
At the start: 471 x 127 mm, 387 parts, among them IC1 REG1117, J1 1-2295018-2, M1 KEYSWITCH-PLAIN-ALPSMX-1U, M2 KEYSWITCH-PLAIN-ALPSMX-1U, M3 KEYSWITCH-PLAIN-ALPSMX-1U, M4 KEYSWITCH-PLAIN-ALPSMX-1U, M5 KEYSWITCH-PLAIN-ALPSMX-1U, M6 KEYSWITCH-PLAIN-ALPSMX-1U

Commit message: Updated Board with matrix
Parts:
- moved DSHIFT2 339.1 mm to (-14.0, -157.0), turned to 0 degrees
- moved J1 148.8 mm to (312.2, 123.4), flipped to the bottom
- moved IC1 122.9 mm to (306.0, 52.0), turned to 0 degrees
- moved U$1 4.12 mm to (321.0, 42.0), turned to 90 degrees
Connections:
- removed net COL22: U$1.6
- removed net N$110: 3.ALPS1, 3.MX1, C.ALPS1, C.MX1, D.ALPS1, D.MX1, E.ALPS1, E.MX1, F3.ALPS1, F3.MX1
- removed net N$112: 4.ALPS1, 4.MX1, F.ALPS1, F.MX1, F4.ALPS1, F4.MX1, R.ALPS1, R.MX1, V.ALPS1, V.MX1
- removed net N$113: 5.ALPS1, 5.MX1, B.ALPS1, B.MX1, F5.ALPS1, F5.MX1, G.ALPS1, G.MX1, SPACE.ALPS1, SPACE.MX1, T.ALPS1, T.MX1
- removed net N$114: 6.ALPS1, 6.MX1, F6.ALPS1, F6.MX1, H.ALPS1, H.MX1, N.ALPS1, N.MX1, Y.ALPS1, Y.MX1
- removed net N$117: 7.ALPS1, 7.MX1, F7.ALPS1, F7.MX1, J.ALPS1, J.MX1, M.ALPS1, M.MX1, U.ALPS1, U.MX1
- removed net N$124: 8.ALPS1, 8.MX1, COMMA.ALPS1, COMMA.MX1, F8.ALPS1, F8.MX1, I.ALPS1, I.MX1, K.ALPS1, K.MX1
- removed net N$125: LKP_DEL.DOUT
- removed net N$127: LBACK.DIN
- removed net N$128: 9.ALPS1, 9.MX1, ALT2.ALPS1, ALT2.MX1, F9.ALPS1, F9.MX1, L.ALPS1, L.MX1, O.ALPS1, O.MX1, PERIOD.ALPS1, PERIOD.MX1
- removed net N$129: 0.ALPS1, 0.MX1, F10.ALPS1, F10.MX1, P.ALPS1, P.MX1, SEMICOLON.ALPS1, SEMICOLON.MX1, SLASH.ALPS1, SLASH.MX1, WIN2.ALPS1, WIN2.MX1
- removed net N$130: DASH.ALPS1, DASH.MX1, F11.ALPS1, F11.MX1, LBRACKET.ALPS1, LBRACKET.MX1, MENU.ALPS1, MENU.MX1, QUOTE.ALPS1, QUOTE.MX1
- removed net N$131: CTRL2.ALPS1, CTRL2.MX1, ENTER.ALPS1, ENTER.MX1, EQUAL.ALPS1, EQUAL.MX1, F12.ALPS1, F12.MX1, RBRACKET.ALPS1, RBRACKET.MX1, SHIFT2.ALPS1, SHIFT2.MX1
- removed net N$132: BACKSLASH.ALPS1, BACKSLASH.MX1, BACKSPACE.ALPS1, BACKSPACE.MX1, VD.ALPS1, VD.MX1, VU.ALPS1, VU.MX1
- removed net N$133: DELETE.ALPS1, DELETE.MX1, INSERT.ALPS1, INSERT.MX1, LEFT.ALPS1, LEFT.MX1, PRTSC.ALPS1, PRTSC.MX1
- removed net N$134: DLAST.C, DLOCK.C, DNEXTSONG.C, DPAUSE.C, DPLAY.C, DPRTSC.C, DRAND.C, DSCROLLLOCK.C
- removed net N$135: DOWN.ALPS1, DOWN.MX1, END.ALPS1, END.MX1, HOME.ALPS1, HOME.MX1, SCROLLLOCK.ALPS1, SCROLLLOCK.MX1, UP.ALPS1, UP.MX1
- removed net N$136: PAUSE.ALPS1, PAUSE.MX1, PGDN.ALPS1, PGDN.MX1, PGUP.ALPS1, PGUP.MX1, RIGHT.ALPS1, RIGHT.MX1
- removed net N$137: KP_2.ALPS1, KP_2.MX1, KP_5.ALPS1, KP_5.MX1, KP_8.ALPS1, KP_8.MX1, KP_DEL.ALPS1, KP_DEL.MX1, KP_SLASH.ALPS1, KP_SLASH.MX1, PLAY.ALPS1, PLAY.MX1
- removed net N$138: KP_0.ALPS1, KP_0.MX1, KP_1.ALPS1, KP_1.MX1, KP_4.ALPS1, KP_4.MX1, KP_7.ALPS1, KP_7.MX1, LAST.ALPS1, LAST.MX1, NUMLOCK.ALPS1, NUMLOCK.MX1
- removed net N$139: KP_3.ALPS1, KP_3.MX1, KP_6.ALPS1, KP_6.MX1, KP_9.ALPS1, KP_9.MX1, KP_ASTERISK.ALPS1, KP_ASTERISK.MX1, NEXTSONG.ALPS1, NEXTSONG.MX1
- removed net N$141: BACK.ALPS1, BACK.MX1, DEL.ALPS1, DEL.MX1, KP_52.ALPS1, KP_52.MX1, KP_62.ALPS1, KP_62.MX1, LOCK.ALPS1, LOCK.MX1, UNDERSCORE.ALPS1, UNDERSCORE.MX1
- removed net N$173: C4.1, C6.1
- removed net N$47: M1.ALPS1, M1.MX1, M2.ALPS1, M2.MX1, M3.ALPS1, M3.MX1, M4.ALPS1, M4.MX1, M5.ALPS1, M5.MX1, M6.ALPS1, M6.MX1
- new net LEDOUT: U$1.18
- net +3V3: now also C4.1, C6.1
- net COL1: now also M1.ALPS1, M1.MX1, M2.ALPS1, M2.MX1, M3.ALPS1, M3.MX1, M4.ALPS1, M4.MX1, M5.ALPS1, M5.MX1, M6.ALPS1, M6.MX1, U$1.5; no longer U$1.18
- net COL10: now also 8.ALPS1, 8.MX1, BACKSLASH.ALPS1, BACKSLASH.MX1, COMMA.ALPS1, COMMA.MX1, F8.ALPS1, F8.MX1, I.ALPS1, I.MX1, K.ALPS1, K.MX1
- net COL11: now also 9.ALPS1, 9.MX1, ALT2.ALPS1, ALT2.MX1, F9.ALPS1, F9.MX1, L.ALPS1, L.MX1, O.ALPS1, O.MX1, PERIOD.ALPS1, PERIOD.MX1
- net COL12: now also 0.ALPS1, 0.MX1, F10.ALPS1, F10.MX1, P.ALPS1, P.MX1, SEMICOLON.ALPS1, SEMICOLON.MX1, SLASH.ALPS1, SLASH.MX1, WIN2.ALPS1, WIN2.MX1
- net COL13: now also DASH.ALPS1, DASH.MX1, F11.ALPS1, F11.MX1, LBRACKET.ALPS1, LBRACKET.MX1, MENU.ALPS1, MENU.MX1, QUOTE.ALPS1, QUOTE.MX1, SHIFT2.ALPS1, SHIFT2.MX1
- net COL14: now also CTRL2.ALPS1, CTRL2.MX1, ENTER.ALPS1, ENTER.MX1, EQUAL.ALPS1, EQUAL.MX1, F12.ALPS1, F12.MX1, RBRACKET.ALPS1, RBRACKET.MX1, VU.ALPS1, VU.MX1
- net COL15: now also DELETE.ALPS1, DELETE.MX1, INSERT.ALPS1, INSERT.MX1, LEFT.ALPS1, LEFT.MX1, PRTSC.ALPS1, PRTSC.MX1, RAND.ALPS1, RAND.MX1
- net COL16: now also DOWN.ALPS1, DOWN.MX1, END.ALPS1, END.MX1, HOME.ALPS1, HOME.MX1, KP_DASH.ALPS1, KP_DASH.MX1, SCROLLLOCK.ALPS1, SCROLLLOCK.MX1, UP.ALPS1, UP.MX1
- net COL17: now also EQUAL2.ALPS1, EQUAL2.MX1, PAUSE.ALPS1, PAUSE.MX1, PGDN.ALPS1, PGDN.MX1, PGUP.ALPS1, PGUP.MX1, RIGHT.ALPS1, RIGHT.MX1
- net COL18: now also KP_0.ALPS1, KP_0.MX1, KP_1.ALPS1, KP_1.MX1, KP_4.ALPS1, KP_4.MX1, KP_7.ALPS1, KP_7.MX1, LAST.ALPS1, LAST.MX1, NUMLOCK.ALPS1, NUMLOCK.MX1
- net COL19: now also KP_2.ALPS1, KP_2.MX1, KP_5.ALPS1, KP_5.MX1, KP_8.ALPS1, KP_8.MX1, KP_DEL.ALPS1, KP_DEL.MX1, KP_SLASH.ALPS1, KP_SLASH.MX1, PLAY.ALPS1, PLAY.MX1
- net COL2: now also CAPSLOCK.ALPS1, CAPSLOCK.MX1, CTRL.ALPS1, CTRL.MX1, ESC.ALPS1, ESC.MX1, GRAVE.ALPS1, GRAVE.MX1, SHIFT.ALPS1, SHIFT.MX1, TAB.ALPS1, TAB.MX1
- net COL20: now also ENTER2.ALPS1, ENTER2.MX1, KP_3.ALPS1, KP_3.MX1, KP_6.ALPS1, KP_6.MX1, KP_9.ALPS1, KP_9.MX1, KP_ASTERISK.ALPS1, KP_ASTERISK.MX1, NEXTSONG.ALPS1, NEXTSONG.MX1
- net COL21: now also BACK.ALPS1, BACK.MX1, DEL.ALPS1, DEL.MX1, KP_52.ALPS1, KP_52.MX1, KP_62.ALPS1, KP_62.MX1, LOCK.ALPS1, LOCK.MX1, U$1.6, UNDERSCORE.ALPS1, UNDERSCORE.MX1; no longer U$1.5
- net COL3: now also 1.ALPS1, 1.MX1, A.ALPS1, A.MX1, F1.ALPS1, F1.MX1, Q.ALPS1, Q.MX1, WIN.ALPS1, WIN.MX1, Z.ALPS1, Z.MX1
- net COL4: now also 2.ALPS1, 2.MX1, ALT.ALPS1, ALT.MX1, F2.ALPS1, F2.MX1, S.ALPS1, S.MX1, W.ALPS1, W.MX1, X.ALPS1, X.MX1
- net COL5: now also 3.ALPS1, 3.MX1, C.ALPS1, C.MX1, D.ALPS1, D.MX1, E.ALPS1, E.MX1, F3.ALPS1, F3.MX1
- net COL6: now also 4.ALPS1, 4.MX1, F.ALPS1, F.MX1, F4.ALPS1, F4.MX1, R.ALPS1, R.MX1, V.ALPS1, V.MX1
- net COL7: now also 5.ALPS1, 5.MX1, B.ALPS1, B.MX1, F5.ALPS1, F5.MX1, G.ALPS1, G.MX1, SPACE.ALPS1, SPACE.MX1, T.ALPS1, T.MX1
- net COL8: now also 6.ALPS1, 6.MX1, F6.ALPS1, F6.MX1, H.ALPS1, H.MX1, N.ALPS1, N.MX1, VD.ALPS1, VD.MX1, Y.ALPS1, Y.MX1
- net COL9: now also 7.ALPS1, 7.MX1, BACKSPACE.ALPS1, BACKSPACE.MX1, F7.ALPS1, F7.MX1, J.ALPS1, J.MX1, M.ALPS1, M.MX1, U.ALPS1, U.MX1
- net N$103: now also DHOME.C, DINSERT.C, DKP_ASTERISK.C, DKP_SLASH.C, DNUMLOCK.C, DPGUP.C, DUNDERSCORE.C; no longer 1.ALPS1, 1.MX1, A.ALPS1, A.MX1, F1.ALPS1, F1.MX1, Q.ALPS1, Q.MX1, WIN.ALPS1, WIN.MX1, Z.ALPS1, Z.MX1
- net N$109: now also DDELETE.C, DEND.C, DKP_52.C, DKP_7.C, DKP_8.C, DKP_9.C, DPGDN.C; no longer 2.ALPS1, 2.MX1, ALT.ALPS1, ALT.MX1, F2.ALPS1, F2.MX1, S.ALPS1, S.MX1, W.ALPS1, W.MX1, X.ALPS1, X.MX1
- net N$84: now also LBACK.DIN, LKP_DEL.DOUT; no longer CAPSLOCK.ALPS1, CAPSLOCK.MX1, CTRL.ALPS1, CTRL.MX1, ESC.ALPS1, ESC.MX1, GRAVE.ALPS1, GRAVE.MX1, SHIFT.ALPS1, SHIFT.MX1, TAB.ALPS1, TAB.MX1
- net ROW1: now also DLAST.C, DLOCK.C, DNEXTSONG.C, DPAUSE.C, DPLAY.C, DPRTSC.C, DSCROLLLOCK.C; no longer DVD.C
- net ROW2: no longer DBACKSPACE.C, DHOME.C, DINSERT.C, DKP_ASTERISK.C, DKP_DASH.C, DKP_SLASH.C, DNUMLOCK.C, DPGUP.C, DUNDERSCORE.C
- net ROW3: no longer DBACKSLASH.C, DDELETE.C, DEND.C, DEQUAL2.C, DKP_52.C, DKP_7.C, DKP_8.C, DKP_9.C, DPGDN.C
- net ROW4: now also DEQUAL2.C, DKP_DASH.C, DRAND.C; no longer DVU.C
- net ROW5: now also DVU.C; no longer DENTER2.C
- net ROW6: now also DENTER2.C, DVD.C

Commit message: Added Initial Routing
Parts:
- removed D11: 4148, Components:SOD-123
- removed R4: 175, rcl:R0603
- added C11: 100nF, rcl:C0402
- added C12: 100nF, rcl:C0805
- added JP1: (no value), pinhead:1X04
- added R5: 5.1k, rcl:R0603
- added VD1: (no value), usblc6:SOT-23-6L
- C1, C2, C3, C4, C5, C6, C7: device rcl:C0805 -> rcl:C0402
- C10: value 22uF -> 10uF
- C9: value 10uF -> 100nF
- R3: value 124 -> 5.1k
- S1: device switch-omron:B3F-31XX -> switch-omron:B3F-10XX
- moved R3 511.0 mm to (450.6, 134.4), turned to 180 degrees
- moved C9 499.5 mm to (437.1, 141.2), turned to 90 degrees
- moved C2 497.6 mm to (399.5, 143.3)
- moved C4 491.9 mm to (407.9, 133.2), turned to 180 degrees
- moved C6 489.2 mm to (399.8, 134.4), turned to 90 degrees
- moved C5 489.2 mm to (412.8, 140.2), turned to 270 degrees
- moved C1 487.0 mm to (414.2, 140.2), turned to 270 degrees
- moved C7 487.0 mm to (399.5, 144.5)
- moved C3 477.4 mm to (398.6, 134.4), turned to 90 degrees
- moved C10 462.3 mm to (429.9, 133.8), turned to 180 degrees
- moved T1 460.0 mm to (412.9, 128.3), turned to 180 degrees
- moved R1 454.9 mm to (410.3, 128.4), turned to 90 degrees
- moved R2 454.2 mm to (407.9, 128.2), turned to 270 degrees
- moved S1 452.9 mm to (400.3, 126.2), turned to 270 degrees
- moved D10 450.6 mm to (409.4, 125.9), turned to 180 degrees
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Connections:
- removed net D+: J1.A6, J1.B6, U$1.33
- removed net D-: J1.A7, J1.B7, U$1.32
- removed net N$172: C9.1, IC1.1, R3.1, R4.2
- new net D+IN: J1.A6, J1.B6, VD1.1
- new net D+OUT: U$1.33, VD1.6
- new net D-IN: J1.A7, J1.B7, VD1.3
- new net D-OUT: U$1.32, VD1.4
- new net N$110: JP1.1, U$1.34
- new net N$112: JP1.2, U$1.37
- net +3V3: now also C11.1, S1.3; no longer D11.A, R3.2, S1.1
- net +5V: now also C12.1, C9.1, VD1.5; no longer D11.C
- net CC1: now also R3.1
- net CC2: now also R5.1
- net GND: now also C11.2, C12.2, IC1.1, JP1.4, R3.2, R5.2, VD1.2; no longer R4.1
- net N$144: now also S1.1; no longer S1.2
- net NRESET: now also JP1.3
Routing:
- net +3V3: track 0.00 -> 82.1 mm, vias 0 -> 1
- net D-OUT: track 0.00 -> 66.9 mm
- net D+OUT: track 0.00 -> 64.9 mm
- net CC2: track 0.00 -> 62.7 mm, vias 0 -> 3
- net CC1: track 0.00 -> 59.9 mm, vias 0 -> 2
- net GND: track 0.00 -> 53.1 mm, vias 0 -> 14
- net +5V: track 0.00 -> 36.0 mm
- net D+IN: track 0.00 -> 18.6 mm, vias 0 -> 2
- net NRESET: track 0.00 -> 17.6 mm, vias 0 -> 2
- net D-IN: track 0.00 -> 15.7 mm, vias 0 -> 2
- net N$144: track 0.00 -> 13.2 mm
- net BOOT0: track 0.00 -> 11.3 mm, vias 0 -> 2
- net N$145: track 0.00 -> 1.69 mm
- added copper zone on layer 16, net GND
Other:
- board size 471 x 127 mm -> 470.5 x 148.6 mm

Commit message: Finished general key routing.
Parts:
- moved J1 155.7 mm to (310.6, 126.5), turned to 180 degrees
- moved C12 151.8 mm to (306.6, 116.8), turned to 180 degrees
- moved C9 150.7 mm to (311.9, 57.4), turned to 180 degrees
- moved C7 146.8 mm to (310.6, 27.7), turned to 90 degrees
- moved R5 146.2 mm to (307.6, 111.3), turned to 270 degrees
- moved IC1 145.4 mm to (314.8, 51.9), turned to 180 degrees
- moved C2 145.2 mm to (311.8, 27.7), turned to 90 degrees
- moved VD1 143.7 mm to (310.9, 113.0), turned to 180 degrees
- moved C5 139.4 mm to (314.9, 40.9), turned to 0 degrees
- moved C1 139.4 mm to (314.9, 42.3), turned to 0 degrees
- moved C10 138.6 mm to (319.3, 50.2), turned to 270 degrees
- moved U$1 138.4 mm to (316.0, 32.7), turned to 270 degrees
- moved R3 137.8 mm to (314.7, 111.3), turned to 270 degrees
- moved C11 133.3 mm to (319.3, 41.1), turned to 90 degrees
- moved C3 132.8 mm to (320.8, 26.8), turned to 180 degrees
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Connections:
- removed net N$103: DHOME.C, DINSERT.C, DKP_ASTERISK.C, DKP_SLASH.C, DNUMLOCK.C, DPGUP.C, DUNDERSCORE.C
- removed net N$109: DDELETE.C, DEND.C, DKP_52.C, DKP_7.C, DKP_8.C, DKP_9.C, DPGDN.C
- net COL1: now also U$1.18; no longer U$1.5
- net COL10: now also 6.ALPS1, 6.MX1, F6.ALPS1, F6.MX1, H.ALPS1, H.MX1, N.ALPS1, N.MX1, U$1.30, Y.ALPS1, Y.MX1; no longer 8.ALPS1, 8.MX1, COMMA.ALPS1, COMMA.MX1, F8.ALPS1, F8.MX1, I.ALPS1, I.MX1, K.ALPS1, K.MX1, U$1.29
- net COL11: now also U$1.29; no longer U$1.30
- net COL12: now also U$1.28; no longer U$1.31
- net COL13: now also U$1.27; no longer U$1.38
- net COL14: now also U$1.26; no longer U$1.39
- net COL15: now also EQUAL2.ALPS1, EQUAL2.MX1, U$1.6; no longer RAND.ALPS1, RAND.MX1, U$1.40
- net COL16: now also U$1.5; no longer U$1.41
- net COL17: now also RAND.ALPS1, RAND.MX1, U$1.45; no longer EQUAL2.ALPS1, EQUAL2.MX1, U$1.42
- net COL19: now also U$1.42; no longer U$1.45
- net COL20: now also U$1.41; no longer U$1.46
- net COL21: now also U$1.40; no longer U$1.6
- net COL7: now also U$1.39; no longer U$1.26
- net COL8: now also 8.ALPS1, 8.MX1, COMMA.ALPS1, COMMA.MX1, F8.ALPS1, F8.MX1, I.ALPS1, I.MX1, K.ALPS1, K.MX1, U$1.38; no longer 6.ALPS1, 6.MX1, F6.ALPS1, F6.MX1, H.ALPS1, H.MX1, N.ALPS1, N.MX1, U$1.27, Y.ALPS1, Y.MX1
- net COL9: now also U$1.31; no longer U$1.28
- net LEDOUT: now also U$1.46; no longer U$1.18
- net ROW2: now also DHOME.C, DINSERT.C, DKP_ASTERISK.C, DKP_SLASH.C, DNUMLOCK.C, DPGUP.C, DUNDERSCORE.C
- net ROW3: now also DDELETE.C, DEND.C, DKP_52.C, DKP_7.C, DKP_8.C, DKP_9.C, DPGDN.C
- net ROW5: no longer DVU.C
- net ROW6: now also DBACKSLASH.C, DBACKSPACE.C, DVU.C
Routing:
- net +5V: track 36.0 -> 2432.9 mm
- net ROW6: track 0.00 -> 665.5 mm, vias 0 -> 10
- net ROW1: track 0.00 -> 519.7 mm, vias 0 -> 4
- net COL1: track 0.00 -> 517.9 mm, vias 0 -> 1
- net COL2: track 0.00 -> 517.8 mm, vias 0 -> 1
- net ROW2: track 0.00 -> 503.7 mm, vias 0 -> 8
- net COL3: track 0.00 -> 502.8 mm, vias 0 -> 1
- net ROW5: track 0.00 -> 491.4 mm, vias 0 -> 2
- net COL4: track 0.00 -> 489.3 mm, vias 0 -> 1
- net ROW3: track 0.00 -> 487.8 mm, vias 0 -> 6
- net COL10: track 0.00 -> 469.4 mm, vias 0 -> 1
- net ROW4: track 0.00 -> 448.3 mm, vias 0 -> 2
- net COL5: track 0.00 -> 444.9 mm, vias 0 -> 1
- net COL9: track 0.00 -> 442.4 mm, vias 0 -> 1
- net COL6: track 0.00 -> 429.3 mm, vias 0 -> 1
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Other:
- board size 470.5 x 148.6 mm -> 479.9 x 132.5 mm

Commit message: Updated Board with power and gnd for leds
Parts:
- moved JP1 82.1 mm to (337.6, 43.4), turned to 270 degrees
- moved S1 71.9 mm to (325.6, 51.8)
- turned L0 to 90 degrees
- turned L1 to 90 degrees
- turned L2 to 90 degrees
- turned L3 to 90 degrees
- turned L4 to 90 degrees
- turned L5 to 90 degrees
- turned L6 to 90 degrees
- turned L7 to 90 degrees
- turned L8 to 90 degrees
- turned L9 to 90 degrees
- turned LA to 90 degrees
- turned LALT to 90 degrees
- turned LALT2 to 90 degrees
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Connections:
- removed net N$126: LKP_0.DOUT, LKP_DEL.DIN
- new net N$103: LKP_52.DOUT, LUNDERSCORE.DIN
- new net N$109: LKP_DASH.DIN, LUNDERSCORE.DOUT
- new net N$113: LM5.DOUT, LM6.DIN
- new net N$114: LBACK.DIN, LLOCK.DOUT
- new net N$117: LCTRL2.DIN, LLEFT.DOUT
- new net N$47: LDEL.DOUT, LKP_62.DIN
- net +3V3: now also S1.4; no longer S1.3
- net COL10: now also U$1.38; no longer U$1.30
- net COL8: now also U$1.30; no longer U$1.38
- net LEDOUT: now also LUP.DIN
- net N$100: now also LALT.DIN, LSPACE.DOUT; no longer LCTRL.DOUT, LWIN.DIN
- net N$101: now also LALT2.DOUT, LSPACE.DIN; no longer LALT.DIN, LWIN.DOUT
- net N$102: now also LKP_6.DIN, LKP_62.DOUT; no longer LSHIFT2.DOUT, LUP.DIN
- net N$111: now also LALT2.DIN, LWIN2.DOUT; no longer LALT.DOUT, LSPACE.DIN
- net N$115: now also LMENU.DOUT, LWIN2.DIN; no longer LALT2.DIN, LSPACE.DOUT
- net N$116: now also LCTRL2.DOUT, LMENU.DIN; no longer LALT2.DOUT, LWIN2.DIN
- net N$118: now also LDOWN.DOUT, LLEFT.DIN; no longer LMENU.DIN, LWIN2.DOUT
- net N$119: now also LDOWN.DIN, LRIGHT.DOUT; no longer LCTRL2.DIN, LMENU.DOUT
- net N$120: now also LKP_0.DOUT, LRIGHT.DIN; no longer LCTRL2.DOUT, LLEFT.DIN
- net N$121: now also LKP_0.DIN, LKP_DEL.DOUT; no longer LDOWN.DIN, LLEFT.DOUT
- net N$122: now also LBACK.DOUT, LKP_DEL.DIN; no longer LDOWN.DOUT, LRIGHT.DIN
- net N$123: now also LM1.DOUT, LM2.DIN; no longer LKP_0.DIN, LRIGHT.DOUT
- net N$144: now also S1.2; no longer S1.1
- net N$24: now also LGRAVE.DOUT, LM5.DIN; no longer LGRAVE.DIN, LM5.DOUT
- net N$25: now also L1.DOUT, LGRAVE.DIN; no longer L1.DIN, LGRAVE.DOUT
- net N$26: now also L1.DIN, L2.DOUT; no longer L1.DOUT, L2.DIN
- net N$27: now also L2.DIN, L3.DOUT; no longer L2.DOUT, L3.DIN
- net N$28: now also L3.DIN, L4.DOUT; no longer L3.DOUT, L4.DIN
- net N$29: now also L4.DIN, L5.DOUT; no longer L4.DOUT, L5.DIN
- net N$30: now also L5.DIN, L6.DOUT; no longer L5.DOUT, L6.DIN
- net N$31: now also L6.DIN, L7.DOUT; no longer L6.DOUT, L7.DIN
- net N$32: now also L7.DIN, L8.DOUT; no longer L7.DOUT, L8.DIN
- net N$33: now also L8.DIN, L9.DOUT; no longer L8.DOUT, L9.DIN
- net N$34: now also L0.DOUT, L9.DIN; no longer L0.DIN, L9.DOUT
- net N$35: now also L0.DIN, LDASH.DOUT; no longer L0.DOUT, LDASH.DIN
- net N$36: now also LDASH.DIN, LEQUAL.DOUT; no longer LDASH.DOUT, LEQUAL.DIN
- net N$38: now also LBACKSPACE.DOUT, LEQUAL.DIN; no longer LBACKSPACE.DIN, LEQUAL.DOUT
- net N$39: now also LCTRL.DOUT, LM1.DIN; no longer LBACKSPACE.DOUT, LINSERT.DIN
- net N$40: now also LBACKSPACE.DIN; no longer LHOME.DIN
- net N$41: now also LINSERT.DIN; no longer LPGUP.DIN
- net N$42: now also LHOME.DIN; no longer LNUMLOCK.DIN
- net N$43: now also LPGUP.DIN; no longer LKP_SLASH.DIN
- net N$44: now also LKP_SLASH.DOUT, LNUMLOCK.DIN; no longer LKP_ASTERISK.DOUT, LKP_DASH.DIN
- net N$45: now also LKP_ASTERISK.DOUT, LKP_SLASH.DIN; no longer LKP_ASTERISK.DIN, LKP_SLASH.DOUT
- net N$46: now also LKP_ASTERISK.DIN; no longer LUNDERSCORE.DIN
- net N$61: now also LM4.DIN; no longer LCAPSLOCK.DIN
- net N$70: now also LM3.DIN; no longer LA.DIN
- net N$71: now also LCAPSLOCK.DIN; no longer LS.DIN
- net N$72: now also LA.DIN; no longer LD.DIN
- net N$73: now also LS.DIN; no longer LF.DIN
- net N$74: now also LD.DIN; no longer LG.DIN
- net N$75: now also LF.DIN; no longer LH.DIN
- net N$76: now also LG.DIN; no longer LJ.DIN
- net N$77: now also LH.DIN; no longer LK.DIN
- net N$78: now also LJ.DIN; no longer LL.DIN
- net N$79: now also LK.DIN; no longer LSEMICOLON.DIN
- net N$80: now also LL.DIN; no longer LQUOTE.DIN
- net N$81: now also LSEMICOLON.DIN; no longer LENTER.DIN
- net N$84: now also LCTRL.DIN, LWIN.DOUT; no longer LBACK.DIN, LKP_DEL.DOUT
- net N$87: now also LQUOTE.DIN; no longer LKP_4.DIN
- net N$88: now also LENTER.DIN; no longer LKP_5.DIN
- net N$90: now also LKP_4.DIN; no longer LKP_6.DIN
- net N$91: now also LKP_5.DIN; no longer LKP_62.DIN
- net N$98: now also LALT.DOUT, LWIN.DIN; no longer LCTRL.DIN, LM1.DOUT
Routing:
- net +5V: track 2432.9 -> 3330.4 mm, vias 0 -> 119
- net N$88: track 0.00 -> 107.7 mm, vias 0 -> 4
- net ROW4: track 448.3 -> 534.6 mm, vias 2 -> 4
- net COL10: track 469.4 -> 528.2 mm
- net N$110: track 0.00 -> 43.3 mm, vias 0 -> 2
- net COL14: track 137.0 -> 179.4 mm
- net N$16: track 0.00 -> 41.6 mm, vias 0 -> 2
- net N$40: track 0.00 -> 39.4 mm, vias 0 -> 2
- net N$62: track 0.00 -> 32.7 mm, vias 0 -> 2
- net N$117: track 0.00 -> 30.3 mm, vias 0 -> 2
- net LEDOUT: track 0.00 -> 28.2 mm, vias 0 -> 1
- net N$112: track 7.30 -> 34.1 mm, vias 0 -> 2
- net COL8: track 428.4 -> 402.9 mm
- net NRESET: track 15.5 -> 34.1 mm, vias 2 -> 3
- net COL9: track 442.4 -> 459.0 mm
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