File: EAGLE_PCB_V2/board.sch (EAGLE design)
At the start: 387 parts, among them IC1 REG1117, J1 1-2295018-2, M1 KEYSWITCH-PLAIN-ALPSMX-1U, M2 KEYSWITCH-PLAIN-ALPSMX-1U, M3 KEYSWITCH-PLAIN-ALPSMX-1U, M4 KEYSWITCH-PLAIN-ALPSMX-1U, M5 KEYSWITCH-PLAIN-ALPSMX-1U, M6 KEYSWITCH-PLAIN-ALPSMX-1U

Commit message: Updated Board with matrix
Connections:
- removed net COL22: U$1.PF1/OSC_OUT
- removed net N$110: 3.P0, C.P0, D.P0, E.P0, F3.P0
- removed net N$112: 4.P0, F.P0, F4.P0, R.P0, V.P0
- removed net N$113: 5.P0, B.P0, F5.P0, G.P0, SPACE.P0, T.P0
- removed net N$114: 6.P0, F6.P0, H.P0, N.P0, Y.P0
- removed net N$117: 7.P0, F7.P0, J.P0, M.P0, U.P0
- removed net N$124: 8.P0, COMMA.P0, F8.P0, I.P0, K.P0
- removed net N$125: LKP_DEL.DOUT
- removed net N$127: LBACK.DIN
- removed net N$128: 9.P0, ALT2.P0, F9.P0, L.P0, O.P0, PERIOD.P0
- removed net N$129: 0.P0, F10.P0, P.P0, SEMICOLON.P0, SLASH.P0, WIN2.P0
- removed net N$130: DASH.P0, F11.P0, LBRACKET.P0, MENU.P0, QUOTE.P0
- removed net N$131: CTRL2.P0, ENTER.P0, EQUAL.P0, F12.P0, RBRACKET.P0, SHIFT2.P0
- removed net N$132: BACKSLASH.P0, BACKSPACE.P0, VD.P0, VU.P0
- removed net N$133: DELETE.P0, INSERT.P0, LEFT.P0, PRTSC.P0
- removed net N$134: DLAST.C, DLOCK.C, DNEXTSONG.C, DPAUSE.C, DPLAY.C, DPRTSC.C, DRAND.C, DSCROLLLOCK.C
- removed net N$135: DOWN.P0, END.P0, HOME.P0, SCROLLLOCK.P0, UP.P0
- removed net N$136: PAUSE.P0, PGDN.P0, PGUP.P0, RIGHT.P0
- removed net N$137: KP_2.P0, KP_5.P0, KP_8.P0, KP_DEL.P0, KP_SLASH.P0, PLAY.P0
- removed net N$138: KP_0.P0, KP_1.P0, KP_4.P0, KP_7.P0, LAST.P0, NUMLOCK.P0
- removed net N$139: KP_3.P0, KP_6.P0, KP_9.P0, KP_ASTERISK.P0, NEXTSONG.P0
- removed net N$141: BACK.P0, DEL.P0, KP_52.P0, KP_62.P0, LOCK.P0, UNDERSCORE.P0
- removed net N$173: C4.1, C6.1
- removed net N$47: M1.P0, M2.P0, M3.P0, M4.P0, M5.P0, M6.P0
- new net LEDOUT: U$1.PB0/ADC_IN8/TIM3_CH3
- net +3V3: now also C4.1, C6.1
- net COL1: now also M1.P0, M2.P0, M3.P0, M4.P0, M5.P0, M6.P0, U$1.PF0/OSC_IN; no longer U$1.PB0/ADC_IN8/TIM3_CH3
- net COL10: now also 8.P0, BACKSLASH.P0, COMMA.P0, F8.P0, I.P0, K.P0
- net COL11: now also 9.P0, ALT2.P0, F9.P0, L.P0, O.P0, PERIOD.P0
- net COL12: now also 0.P0, F10.P0, P.P0, SEMICOLON.P0, SLASH.P0, WIN2.P0
- net COL13: now also DASH.P0, F11.P0, LBRACKET.P0, MENU.P0, QUOTE.P0, SHIFT2.P0
- net COL14: now also CTRL2.P0, ENTER.P0, EQUAL.P0, F12.P0, RBRACKET.P0, VU.P0
- net COL15: now also DELETE.P0, INSERT.P0, LEFT.P0, PRTSC.P0, RAND.P0
- net COL16: now also DOWN.P0, END.P0, HOME.P0, KP_DASH.P0, SCROLLLOCK.P0, UP.P0
- net COL17: now also EQUAL2.P0, PAUSE.P0, PGDN.P0, PGUP.P0, RIGHT.P0
- net COL18: now also KP_0.P0, KP_1.P0, KP_4.P0, KP_7.P0, LAST.P0, NUMLOCK.P0
- net COL19: now also KP_2.P0, KP_5.P0, KP_8.P0, KP_DEL.P0, KP_SLASH.P0, PLAY.P0
- net COL2: now also CAPSLOCK.P0, CTRL.P0, ESC.P0, GRAVE.P0, SHIFT.P0, TAB.P0
- net COL20: now also ENTER2.P0, KP_3.P0, KP_6.P0, KP_9.P0, KP_ASTERISK.P0, NEXTSONG.P0
- net COL21: now also BACK.P0, DEL.P0, KP_52.P0, KP_62.P0, LOCK.P0, U$1.PF1/OSC_OUT, UNDERSCORE.P0; no longer U$1.PF0/OSC_IN
- net COL3: now also 1.P0, A.P0, F1.P0, Q.P0, WIN.P0, Z.P0
- net COL4: now also 2.P0, ALT.P0, F2.P0, S.P0, W.P0, X.P0
- net COL5: now also 3.P0, C.P0, D.P0, E.P0, F3.P0
- net COL6: now also 4.P0, F.P0, F4.P0, R.P0, V.P0
- net COL7: now also 5.P0, B.P0, F5.P0, G.P0, SPACE.P0, T.P0
- net COL8: now also 6.P0, F6.P0, H.P0, N.P0, VD.P0, Y.P0
- net COL9: now also 7.P0, BACKSPACE.P0, F7.P0, J.P0, M.P0, U.P0
- net N$103: now also DHOME.C, DINSERT.C, DKP_ASTERISK.C, DKP_SLASH.C, DNUMLOCK.C, DPGUP.C, DUNDERSCORE.C; no longer 1.P0, A.P0, F1.P0, Q.P0, WIN.P0, Z.P0
- net N$109: now also DDELETE.C, DEND.C, DKP_52.C, DKP_7.C, DKP_8.C, DKP_9.C, DPGDN.C; no longer 2.P0, ALT.P0, F2.P0, S.P0, W.P0, X.P0
- net N$84: now also LBACK.DIN, LKP_DEL.DOUT; no longer CAPSLOCK.P0, CTRL.P0, ESC.P0, GRAVE.P0, SHIFT.P0, TAB.P0
- net ROW1: now also DLAST.C, DLOCK.C, DNEXTSONG.C, DPAUSE.C, DPLAY.C, DPRTSC.C, DSCROLLLOCK.C; no longer DVD.C
- net ROW2: no longer DBACKSPACE.C, DHOME.C, DINSERT.C, DKP_ASTERISK.C, DKP_DASH.C, DKP_SLASH.C, DNUMLOCK.C, DPGUP.C, DUNDERSCORE.C
- net ROW3: no longer DBACKSLASH.C, DDELETE.C, DEND.C, DEQUAL2.C, DKP_52.C, DKP_7.C, DKP_8.C, DKP_9.C, DPGDN.C
- net ROW4: now also DEQUAL2.C, DKP_DASH.C, DRAND.C; no longer DVU.C
- net ROW5: now also DVU.C; no longer DENTER2.C
- net ROW6: now also DENTER2.C, DVD.C
Other:
- moved on the sheet: DSHIFT2, SHIFT2

Commit message: Added Initial Routing
Parts:
- removed D11: 4148, Components:DIODE-SOD-123
- removed R4: 175, rcl:R-EU_R0603
- added C11: 100nF, rcl:C-EUC0402
- added C12: 100nF, rcl:C-EUC0805
- added JP1: (no value), pinhead:PINHD-1X4
- added R5: 5.1k, rcl:R-EU_R0603
- added VD1: (no value), usblc6:USBLC6-2SC6
- C1, C2, C3, C4, C5, C6, C7: device rcl:C-EUC0805 -> rcl:C-EUC0402
- C10: value 22uF -> 10uF
- C9: value 10uF -> 100nF
- R3: value 124 -> 5.1k
- S1: device switch-omron:31-XX -> switch-omron:10-XX
Connections:
- removed net D+: J1.D+, J1.D+@1, U$1.PA12/USB_DP/CAN_TX
- removed net D-: J1.D-, J1.D-@1, U$1.PA11/USB_DM/CAN_RX
- removed net N$172: C9.1, IC1.GND, R3.1, R4.2
- new net D+IN: J1.D+, J1.D+@1, VD1.I/O_1
- new net D+OUT: U$1.PA12/USB_DP/CAN_TX, VD1.I/O1
- new net D-IN: J1.D-, J1.D-@1, VD1.I/O_2
- new net D-OUT: U$1.PA11/USB_DM/CAN_RX, VD1.I/O2
- new net N$110: JP1.1, U$1.PA13/SWDIO
- new net N$112: JP1.2, U$1.PA14/USART2_TX/SWCLK
- net +3V3: now also C11.1; no longer D11.A, R3.2
- net +5V: now also C12.1, C9.1, VD1.VBUS; no longer D11.C
- net CC1: now also R3.1
- net CC2: now also R5.1
- net GND: now also C11.2, C12.2, IC1.GND, JP1.4, R3.2, R5.2, VD1.GND; no longer R4.1
- net NRESET: now also JP1.3
Other:
- moved on the sheet: C10, C2, C3, C4, C6, C7, C8, C9, D10, IC1, R1, R2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

Commit message: Finished general key routing.
Connections:
- removed net N$103: DHOME.C, DINSERT.C, DKP_ASTERISK.C, DKP_SLASH.C, DNUMLOCK.C, DPGUP.C, DUNDERSCORE.C
- removed net N$109: DDELETE.C, DEND.C, DKP_52.C, DKP_7.C, DKP_8.C, DKP_9.C, DPGDN.C
- net COL1: now also U$1.PB0/ADC_IN8/TIM3_CH3; no longer U$1.PF0/OSC_IN
- net COL10: now also 6.P0, F6.P0, H.P0, N.P0, U$1.PA9/USART1_TX/TIM1_CH2, Y.P0; no longer 8.P0, COMMA.P0, F8.P0, I.P0, K.P0, U$1.PA8/TIM1_CH1
- net COL11: now also U$1.PA8/TIM1_CH1; no longer U$1.PA9/USART1_TX/TIM1_CH2
- net COL12: now also U$1.PB15/WKUP7/RTC_REFIN/SPI2_MOSI; no longer U$1.PA10/USART1_RX/TIM1_CH3
- net COL13: now also U$1.PB14/SPI2_MISO/I2C2_SDA; no longer U$1.PA15/USART2_RX
- net COL14: now also U$1.PB13/SPI2_SCK/I2C2_SCL; no longer U$1.PB3/SPI1_SCK/TIM2_CH2
- net COL15: now also EQUAL2.P0, U$1.PF1/OSC_OUT; no longer RAND.P0, U$1.PB4/SPI1_MISO/TIM3_CH1
- net COL16: now also U$1.PF0/OSC_IN; no longer U$1.PB5/WKUP6/SPI1_MOSI/TIM3_CH2
- net COL17: now also RAND.P0, U$1.PB8/I2C1_SCL/TIM16_CH1/CAN_RX; no longer EQUAL2.P0, U$1.PB6USART1_TX/I2C1_SCL
- net COL19: now also U$1.PB6USART1_TX/I2C1_SCL; no longer U$1.PB8/I2C1_SCL/TIM16_CH1/CAN_RX
- net COL20: now also U$1.PB5/WKUP6/SPI1_MOSI/TIM3_CH2; no longer U$1.PB9/I2C1_SDA/TIM17_CH1/CAN_TX
- net COL21: now also U$1.PB4/SPI1_MISO/TIM3_CH1; no longer U$1.PF1/OSC_OUT
- net COL7: now also U$1.PB3/SPI1_SCK/TIM2_CH2; no longer U$1.PB13/SPI2_SCK/I2C2_SCL
- net COL8: now also 8.P0, COMMA.P0, F8.P0, I.P0, K.P0, U$1.PA15/USART2_RX; no longer 6.P0, F6.P0, H.P0, N.P0, U$1.PB14/SPI2_MISO/I2C2_SDA, Y.P0
- net COL9: now also U$1.PA10/USART1_RX/TIM1_CH3; no longer U$1.PB15/WKUP7/RTC_REFIN/SPI2_MOSI
- net LEDOUT: now also U$1.PB9/I2C1_SDA/TIM17_CH1/CAN_TX; no longer U$1.PB0/ADC_IN8/TIM3_CH3
- net ROW2: now also DHOME.C, DINSERT.C, DKP_ASTERISK.C, DKP_SLASH.C, DNUMLOCK.C, DPGUP.C, DUNDERSCORE.C
- net ROW3: now also DDELETE.C, DEND.C, DKP_52.C, DKP_7.C, DKP_8.C, DKP_9.C, DPGDN.C
- net ROW5: no longer DVU.C
- net ROW6: now also DBACKSLASH.C, DBACKSPACE.C, DVU.C

Commit message: Updated Board with power and gnd for leds
Connections:
- removed net N$126: LKP_0.DOUT, LKP_DEL.DIN
- new net N$103: LKP_52.DOUT, LUNDERSCORE.DIN
- new net N$109: LKP_DASH.DIN, LUNDERSCORE.DOUT
- new net N$113: LM5.DOUT, LM6.DIN
- new net N$114: LBACK.DIN, LLOCK.DOUT
- new net N$117: LCTRL2.DIN, LLEFT.DOUT
- new net N$47: LDEL.DOUT, LKP_62.DIN
- net +3V3: now also S1.P1; no longer S1.P
- net COL10: now also U$1.PA15/USART2_RX; no longer U$1.PA9/USART1_TX/TIM1_CH2
- net COL8: now also U$1.PA9/USART1_TX/TIM1_CH2; no longer U$1.PA15/USART2_RX
- net LEDOUT: now also LUP.DIN
- net N$100: now also LALT.DIN, LSPACE.DOUT; no longer LCTRL.DOUT, LWIN.DIN
- net N$101: now also LALT2.DOUT, LSPACE.DIN; no longer LALT.DIN, LWIN.DOUT
- net N$102: now also LKP_6.DIN, LKP_62.DOUT; no longer LSHIFT2.DOUT, LUP.DIN
- net N$111: now also LALT2.DIN, LWIN2.DOUT; no longer LALT.DOUT, LSPACE.DIN
- net N$115: now also LMENU.DOUT, LWIN2.DIN; no longer LALT2.DIN, LSPACE.DOUT
- net N$116: now also LCTRL2.DOUT, LMENU.DIN; no longer LALT2.DOUT, LWIN2.DIN
- net N$118: now also LDOWN.DOUT, LLEFT.DIN; no longer LMENU.DIN, LWIN2.DOUT
- net N$119: now also LDOWN.DIN, LRIGHT.DOUT; no longer LCTRL2.DIN, LMENU.DOUT
- net N$120: now also LKP_0.DOUT, LRIGHT.DIN; no longer LCTRL2.DOUT, LLEFT.DIN
- net N$121: now also LKP_0.DIN, LKP_DEL.DOUT; no longer LDOWN.DIN, LLEFT.DOUT
- net N$122: now also LBACK.DOUT, LKP_DEL.DIN; no longer LDOWN.DOUT, LRIGHT.DIN
- net N$123: now also LM1.DOUT, LM2.DIN; no longer LKP_0.DIN, LRIGHT.DOUT
- net N$144: now also S1.S1; no longer S1.S
- net N$24: now also LGRAVE.DOUT, LM5.DIN; no longer LGRAVE.DIN, LM5.DOUT
- net N$25: now also L1.DOUT, LGRAVE.DIN; no longer L1.DIN, LGRAVE.DOUT
- net N$26: now also L1.DIN, L2.DOUT; no longer L1.DOUT, L2.DIN
- net N$27: now also L2.DIN, L3.DOUT; no longer L2.DOUT, L3.DIN
- net N$28: now also L3.DIN, L4.DOUT; no longer L3.DOUT, L4.DIN
- net N$29: now also L4.DIN, L5.DOUT; no longer L4.DOUT, L5.DIN
- net N$30: now also L5.DIN, L6.DOUT; no longer L5.DOUT, L6.DIN
- net N$31: now also L6.DIN, L7.DOUT; no longer L6.DOUT, L7.DIN
- net N$32: now also L7.DIN, L8.DOUT; no longer L7.DOUT, L8.DIN
- net N$33: now also L8.DIN, L9.DOUT; no longer L8.DOUT, L9.DIN
- net N$34: now also L0.DOUT, L9.DIN; no longer L0.DIN, L9.DOUT
- net N$35: now also L0.DIN, LDASH.DOUT; no longer L0.DOUT, LDASH.DIN
- net N$36: now also LDASH.DIN, LEQUAL.DOUT; no longer LDASH.DOUT, LEQUAL.DIN
- net N$38: now also LBACKSPACE.DOUT, LEQUAL.DIN; no longer LBACKSPACE.DIN, LEQUAL.DOUT
- net N$39: now also LCTRL.DOUT, LM1.DIN; no longer LBACKSPACE.DOUT, LINSERT.DIN
- net N$40: now also LBACKSPACE.DIN; no longer LHOME.DIN
- net N$41: now also LINSERT.DIN; no longer LPGUP.DIN
- net N$42: now also LHOME.DIN; no longer LNUMLOCK.DIN
- net N$43: now also LPGUP.DIN; no longer LKP_SLASH.DIN
- net N$44: now also LKP_SLASH.DOUT, LNUMLOCK.DIN; no longer LKP_ASTERISK.DOUT, LKP_DASH.DIN
- net N$45: now also LKP_ASTERISK.DOUT, LKP_SLASH.DIN; no longer LKP_ASTERISK.DIN, LKP_SLASH.DOUT
- net N$46: now also LKP_ASTERISK.DIN; no longer LUNDERSCORE.DIN
- net N$61: now also LM4.DIN; no longer LCAPSLOCK.DIN
- net N$70: now also LM3.DIN; no longer LA.DIN
- net N$71: now also LCAPSLOCK.DIN; no longer LS.DIN
- net N$72: now also LA.DIN; no longer LD.DIN
- net N$73: now also LS.DIN; no longer LF.DIN
- net N$74: now also LD.DIN; no longer LG.DIN
- net N$75: now also LF.DIN; no longer LH.DIN
- net N$76: now also LG.DIN; no longer LJ.DIN
- net N$77: now also LH.DIN; no longer LK.DIN
- net N$78: now also LJ.DIN; no longer LL.DIN
- net N$79: now also LK.DIN; no longer LSEMICOLON.DIN
- net N$80: now also LL.DIN; no longer LQUOTE.DIN
- net N$81: now also LSEMICOLON.DIN; no longer LENTER.DIN
- net N$84: now also LCTRL.DIN, LWIN.DOUT; no longer LBACK.DIN, LKP_DEL.DOUT
- net N$87: now also LQUOTE.DIN; no longer LKP_4.DIN
- net N$88: now also LENTER.DIN; no longer LKP_5.DIN
- net N$90: now also LKP_4.DIN; no longer LKP_6.DIN
- net N$91: now also LKP_5.DIN; no longer LKP_62.DIN
- net N$98: now also LALT.DOUT, LWIN.DIN; no longer LCTRL.DIN, LM1.DOUT
Other:
- moved on the sheet: L0, L1, L2, L3, L4, L5, L6, L7, L8, L9, LA, LALT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
